File: Energy_Meter.recovered.2026-06-18_162926.kicad_sch (KiCad schematic)
At the start: 51 parts, among them J1 Conn_Jack_Stereo_3.5mm_SMD_RA, J3 USB_C_Receptacle, J5 Conn_01x01_Shielded, J6 Conn_01x01_Shielded, SW1 SW_Push, T2 ZMPT101B, U1 STM32F103C8Tx, U2 INA238, U3 IP5306, U4 AMS1117-3.3

Commit message: update 18/06/2026
Parts:
- added C14: 0.1uF, PCM_SparkFun-Capacitor:C_0603_1608Metric, symbol PCM_SparkFun-Capacitor:0.1uF_0603_100V_10%
- added J7, J8: Conn_01x01_Shielded, symbol Connector_Generic_Shielded:Conn_01x01_Shielded
- added R14, R5: 10, PCM_SparkFun-Resistor:R_1206_3216Metric, symbol PCM_SparkFun-Resistor:10_1206
- added R15_Shunt: 0.001_1%_5W, WSLF25121L000FEA:RESC6331X88N, symbol WSLF25121L000FEA:WSLF25121L000FEA
Connections:
- net SCL: now reaches R12.1, U2.5 (SCL)
- net SCL: now also U1.42 (PB6)
- net SDA: now reaches R11.1, U2.4 (SDA)
- net SDA: now also U1.43 (PB7)
- net IN+: now reaches U2.10 (Vin+)
- net IN+: now also C14.1, J7.1 (Pin_1), R5.2
- net IN-: now reaches U2.8 (Vbus)
- net IN-: now also U2.9 (Vin-), C14.2, J8.1 (Pin_1), R14.2
- new net: R15_Shunt.2, R5.1
- new net: R14.1, R15_Shunt.1
- no-connect marks 5 -> 7
Other:
- moved on the sheet: U1

Commit message: update 18/06/2026
Parts:
- added C15, C16, C17, C18, C19: 100nF_0603_16V, 4ms_Capacitor:C_0603, symbol PCM_4ms_Capacitor:100nF_0603_16V
- added C20, C21: 10nF_0603_25V, 4ms_Capacitor:C_0603, symbol PCM_4ms_Capacitor:10nF_0603_25V
- added C22, C23: 1uF_0603_25V, 4ms_Capacitor:C_0603, symbol PCM_4ms_Capacitor:1uF_0603_25V
- added FB1: FerriteBead, symbol Device:FerriteBead
- added J2: Conn_01x04_Socket, symbol Connector:Conn_01x04_Socket
- added R15, R26: 10k, Resistor_THT:R_Axial_DIN0207_L6.3mm_D2.5mm_P10.16mm_Horizontal, symbol PCM_SL_Resistors:10k
- added R25: 1.5k_0603, 4ms_Resistor:R_0603, symbol PCM_4ms_Resistor:1.5k_0603
- added SW2: Switch_Tactile_CnK, PCM_fab:Button_CnK_PTS636.0_6x3.5mm, symbol PCM_fab:Switch_Tactile_CnK
- added SW3: SW_SPDT, symbol Switch:SW_SPDT
- added U5: DM-OLED096-636, DM-OLED096-636:MODULE_DM-OLED096-636, symbol DM-OLED096-636:DM-OLED096-636
Connections:
- net 3.3V: now also U1.1 (VBAT), U1.24 (VDD), U1.36 (VDD), U1.48 (VDD), C16.1, C17.1, C18.1, C19.1, C20.1, C22.1, FB1.2, J2.1 (Pin_1), R15.1, R25.1, SW3.3 (C), U5.2 (VCC_IN)
- net GND: now also U1.23 (VSS), U1.35 (VSS), U1.47 (VSS), U1.8 (VSSA), C15.2, C16.2, C17.2, C18.2, C19.2, C20.2, C21.1, C22.2, C23.2, J2.4 (Pin_4), SW2.1, SW3.1 (A), U5.1 (GND)
- net USB_C+: now reaches J3.A6 (D+), J3.B6 (D+)
- net USB_C+: now also U1.33 (PA12), R25.2
- net USB_C-: now reaches J3.A7 (D-), J3.B7 (D-)
- net USB_C-: now also U1.32 (PA11)
- net SCL2: now reaches U1.21 (PB10)
- net SCL2: now also U5.3 (SCL)
- net SDA2: now reaches U1.22 (PB11)
- net SDA2: now also U5.4 (SDA)
- net SWDIO: now reaches U1.34 (PA13)
- net SWDIO: now also J2.2 (Pin_2)
- net SWCLK: now reaches U1.37 (PA14)
- net SWCLK: now also J2.3 (Pin_3)
- net at U1.44 (BOOT0): now also R26.2
- net at U1.7 (NRST): now also C15.1, R15.2, SW2.2
- net 3.3VA: now reaches U1.9 (VDDA)
- net 3.3VA: now also C21.2, C23.1, FB1.1
- net SCL renamed SCL1
- net SDA renamed SDA1
- new net: R26.1, SW3.2 (B)
- no-connect marks 7 -> 5
Other:
- moved on the sheet: C12, C13, C14, C8, D6, J1, J7, J8, R10, R11, R12, R13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

Commit message: update 19/06/2026
Other:
- note added: "Khôí hiển thị"
- note added: "Khôí vi điều khiển"
- note added: "Khôí đo dòng, áp, công suất DC"
- note added: "Khối Nguồn"
- note added: "Khối đo dòng AC"
- note added: "Khối đo áp AC"
- moved on the sheet: C15, C16, C17, C18, C19, C20, C21, C22, C23, FB1, J2, R15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

Commit message: update 23/06/2026
Parts:
- removed C23: 1uF_0603_25V, 4ms_Capacitor:C_0603, symbol PCM_4ms_Capacitor:1uF_0603_25V
- removed C5: 10 uF, Capacitor_SMD:C_1206_3216Metric_Pad1.33x1.80mm_HandSolder, symbol Device:C
- removed R6: 2Ω, Resistor_SMD:R_1206_3216Metric, symbol Device:R_US
- removed U3: IP5306, Package_SO:SOP-8-1EP_4.57x4.57mm_P1.27mm_EP4.57x4.45mm_ThermalVias, symbol IP5306:IP5306
- added C23, C25: 100nF_Ceramic, Capacitor_THT:C_Disc_D5.0mm_W2.5mm_P2.50mm, symbol PCM_SL_Capacitors:100nF_Ceramic
- added C24: 10uF_16V, Capacitor_THT:CP_Radial_D5.0mm_P2.00mm, symbol PCM_SL_Capacitors:10uF_16V
- added C5: 10uF, PCM_SparkFun-Capacitor:C_1210_3225Metric, symbol PCM_SparkFun-Capacitor:10uF_1210_50V_20%
- added R27: 10k, Resistor_THT:R_Axial_DIN0207_L6.3mm_D2.5mm_P10.16mm_Horizontal, symbol PCM_SL_Resistors:10k
- added R6: 2, PCM_fab:R_1206, symbol PCM_fab:R_1206
- added U6: IP5306, Components_Footprint:SOP127P600X165-9N, symbol IP5306:IP5306
- C12: footprint 4ms_Capacitor:C_0603 -> PCM_4ms_Capacitor:C_0603
- R15_Shunt1: renamed from R15_Shunt; footprint WSLF25121L000FEA:RESC6331X88N -> Components_Footprint:RESC6331X88N
- R16, R17, R18, R19, R20, R21: footprint ERA8ARB203V:RES_ERA8ARB203V -> Components_Footprint:RES_ERA8ARB203V
- R4_Burden1: renamed from R4; footprint RC1206FR-07360RL:RESC3116X65N -> Components_Footprint:RESC3116X65N
- SW3: footprint (none) -> Components_Footprint:SOP127P600X165-9N
- T2: footprint ZMPT101B:XFMR_ZMPT101B -> Components_Footprint:XFMR_ZMPT101B
- U5: footprint DM-OLED096-636:MODULE_DM-OLED096-636 -> Components_Footprint:MODULE_DM-OLED096-636
Connections:
- net 3.3VA: now also R22.2, R7.2, C23.2
- net 5V: now also C24.1, C25.2, U6.8 (VOUT)
- net BAT: now also R6.1, U6.6 (BAT)
- net GND: now also C23.1, C24.2, C25.1, C5.2, R27.1, U6.9 (GND)
- net VBUS: now also U6.1 (VIN)
- net at D3.2 (A), D4.1 (K): now also U6.3 (LED2)
- net at D1.1 (K), D2.2 (A), D3.1 (K)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: now also U6.4 (LED3)
- net at D1.2 (A), D2.1 (K): now also U6.2 (LED1)
- net at SW1.2: now also U6.5 (KEY)
- net at L1.1: now also U6.7 (SW)
- net at U1.20 (PB2): now also R27.2
- net 3.3V renamed 3.3VD
- net 3.3VD: no longer R22.2, R7.2
- new net: C5.1, R6.2
- no-connect marks 5 -> 31
Other:
- note added: "Khối Nguồn và Bootloader"
- note added: "Khối hiển thị"
- note added: "Khối vi điều khiển"
- note added: "Khối đo dòng, áp, công suất DC"
- note removed: "Khôí hiển thị"
- note removed: "Khôí vi điều khiển"
- note removed: "Khôí đo dòng, áp, công suất DC"
- note removed: "Khối Nguồn"
- moved on the sheet: C10, C2, C3, C4, C9, D1, D2, D3, D4, R26, R3, SW1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

Commit message: update 23/06/2026
Parts:
- removed T2: ZMPT101B, Components_Footprint:XFMR_ZMPT101B, symbol ZMPT101B:ZMPT101B
- added T1: ZMPT101B, Components_Footprint:XFMR_ZMPT101B, symbol ZMPT101B:ZMPT101B
- C1, C2, C3, C4, C6, C7: footprint Capacitor_SMD:C_1206_3216Metric_Pad1.33x1.80mm_HandSolder -> Capacitor_SMD:C_1206_3216Metric
- C13, C15, C16, C17, C18, C19, C20, C21, C22: footprint 4ms_Capacitor:C_0603 -> Capacitor_SMD:C_0603_1608Metric
- FB1: footprint (none) -> Components_Footprint:XFMR_ZMPT101B
- J2: footprint (none) -> Connector_PinSocket_1.00mm:PinSocket_1x04_P1.00mm_Vertical
- J5, J6, J7, J8: footprint (none) -> Connector:Banana_Jack_1Pin
- R16, R17, R18, R19, R20, R21: MANUFACTURER Panasonic -> (none); Manufacturer (none) -> Panasonic
- R25: footprint 4ms_Resistor:R_0603 -> Capacitor_SMD:C_0603_1608Metric
- U5: MANUFACTURER Displaymodule -> (none); Manufacturer (none) -> Displaymodule
Connections:
- net at C11.1, R22.1, R23.2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: now also T1.4
- net at R17.2: now also T1.2
- net at R16.2: now also T1.1
- net at R24.1, R4_Burden1.2: now also T1.3

Commit message: update 23/06/2026
Parts:
- removed R10: 33, PCM_fab:R_1206, symbol PCM_fab:R_1206
- added R10: 33_0805, Components_Footprint:RESC2012X60N, symbol RS73G2ATTD33R0B:RS73G2ATTD33R0B
Connections:
- net at J1.2, R9.1: now also R10.1
- net at C8.1, J1.1, R7.1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: now also R10.2
Other:
- moved on the sheet: D6, R9
