File: Energy_Meter.kicad_sch (KiCad schematic)
At the start: 51 parts, among them J1 Conn_Jack_Stereo_3.5mm_SMD_RA, J3 USB_C_Receptacle, J5 Conn_01x01_Shielded, J6 Conn_01x01_Shielded, SW1 SW_Push, T2 ZMPT101B, U1 STM32F103C8Tx, U2 INA238, U3 IP5306, U4 AMS1117-3.3

Commit message: update 23/06/2026
Parts:
- removed C5: 10 uF, Capacitor_SMD:C_1206_3216Metric_Pad1.33x1.80mm_HandSolder, symbol Device:C
- removed R10: 33, PCM_fab:R_1206, symbol PCM_fab:R_1206
- removed R6: 2Ω, Resistor_SMD:R_1206_3216Metric, symbol Device:R_US
- removed T2: ZMPT101B, ZMPT101B:XFMR_ZMPT101B, symbol ZMPT101B:ZMPT101B
- removed U3: IP5306, Package_SO:SOP-8-1EP_4.57x4.57mm_P1.27mm_EP4.57x4.45mm_ThermalVias, symbol IP5306:IP5306
- added C14: 0.1uF, PCM_SparkFun-Capacitor:C_0603_1608Metric, symbol PCM_SparkFun-Capacitor:0.1uF_0603_100V_10%
- added C15, C16, C17, C18, C19: 100nF_0603_16V, Capacitor_SMD:C_0603_1608Metric, symbol PCM_4ms_Capacitor:100nF_0603_16V
- added C20, C21: 10nF_0603_25V, Capacitor_SMD:C_0603_1608Metric, symbol PCM_4ms_Capacitor:10nF_0603_25V
- added C22: 1uF_0603_25V, Capacitor_SMD:C_0603_1608Metric, symbol PCM_4ms_Capacitor:1uF_0603_25V
- added C23, C25: 100nF_Ceramic, Capacitor_THT:C_Disc_D5.0mm_W2.5mm_P2.50mm, symbol PCM_SL_Capacitors:100nF_Ceramic
- added C24: 10uF_16V, Capacitor_THT:CP_Radial_D5.0mm_P2.00mm, symbol PCM_SL_Capacitors:10uF_16V
- added C5: 10uF, PCM_SparkFun-Capacitor:C_1210_3225Metric, symbol PCM_SparkFun-Capacitor:10uF_1210_50V_20%
- added FB1: FerriteBead, Components_Footprint:XFMR_ZMPT101B, symbol Device:FerriteBead
- added J2: Conn_01x04_Socket, Connector_PinSocket_1.00mm:PinSocket_1x04_P1.00mm_Vertical, symbol Connector:Conn_01x04_Socket
- added J7, J8: Conn_01x01_Shielded, Connector:Banana_Jack_1Pin, symbol Connector_Generic_Shielded:Conn_01x01_Shielded
- added R10: 33_0805, Components_Footprint:RESC2012X60N, symbol RS73G2ATTD33R0B:RS73G2ATTD33R0B
- added R14, R5: 10, PCM_SparkFun-Resistor:R_1206_3216Metric, symbol PCM_SparkFun-Resistor:10_1206
- added R15, R26, R27: 10k, Resistor_THT:R_Axial_DIN0207_L6.3mm_D2.5mm_P10.16mm_Horizontal, symbol PCM_SL_Resistors:10k
- added R15_Shunt1: 0.001_1%_5W, Components_Footprint:RESC6331X88N, symbol WSLF25121L000FEA:WSLF25121L000FEA
- added R25: 1.5k_0603, Capacitor_SMD:C_0603_1608Metric, symbol PCM_4ms_Resistor:1.5k_0603
- added R6: 2, PCM_fab:R_1206, symbol PCM_fab:R_1206
- added SW2: Switch_Tactile_CnK, PCM_fab:Button_CnK_PTS636.0_6x3.5mm, symbol PCM_fab:Switch_Tactile_CnK
- added SW3: SW_SPDT, Components_Footprint:SOP127P600X165-9N, symbol Switch:SW_SPDT
- added T1: ZMPT101B, Components_Footprint:XFMR_ZMPT101B, symbol ZMPT101B:ZMPT101B
- added U5: DM-OLED096-636, Components_Footprint:MODULE_DM-OLED096-636, symbol DM-OLED096-636:DM-OLED096-636
- added U6: IP5306, Components_Footprint:SOP127P600X165-9N, symbol IP5306:IP5306
- C1, C2, C3, C4, C6, C7: footprint Capacitor_SMD:C_1206_3216Metric_Pad1.33x1.80mm_HandSolder -> Capacitor_SMD:C_1206_3216Metric
- C12: footprint 4ms_Capacitor:C_0603 -> PCM_4ms_Capacitor:C_0603
- C13: footprint 4ms_Capacitor:C_0603 -> Capacitor_SMD:C_0603_1608Metric
- J5, J6: footprint (none) -> Connector:Banana_Jack_1Pin
- R16, R17, R18, R19, R20, R21: footprint ERA8ARB203V:RES_ERA8ARB203V -> Components_Footprint:RES_ERA8ARB203V; MANUFACTURER Panasonic -> (none); Manufacturer (none) -> Panasonic
- R4_Burden1: renamed from R4; footprint RC1206FR-07360RL:RESC3116X65N -> Components_Footprint:RESC3116X65N
Connections:
- net 5V: now also C24.1, C25.2, U6.8 (VOUT)
- net BAT: now also R6.1, U6.6 (BAT)
- net GND: now also U1.23 (VSS), U1.35 (VSS), U1.47 (VSS), U1.8 (VSSA), C15.2, C16.2, C17.2, C18.2, C19.2, C20.2, C21.1, C22.2, C23.1, C24.2, C25.1, C5.2, J2.4 (Pin_4), R27.1, SW2.1, SW3.1 (A), U5.1 (GND), U6.9 (GND)
- net VBUS: now also U6.1 (VIN)
- net at D3.2 (A), D4.1 (K): now also U6.3 (LED2)
- net at D1.1 (K), D2.2 (A), D3.1 (K)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: now also U6.4 (LED3)
- net at C11.1, R22.1, R23.2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: now also T1.4
- net at J1.2, R9.1: now also R10.1
- net at D1.2 (A), D2.1 (K): now also U6.2 (LED1)
- net at SW1.2: now also U6.5 (KEY)
- net at L1.1: now also U6.7 (SW)
- net at R17.2: now also T1.2
- net at C8.1, J1.1, R7.1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: now also R10.2
- net at R16.2: now also T1.1
- net at R24.1, R4_Burden1.2: now also T1.3
- net USB_C+: now reaches J3.A6 (D+), J3.B6 (D+)
- net USB_C+: now also U1.33 (PA12), R25.2
- net USB_C-: now reaches J3.A7 (D-), J3.B7 (D-)
- net USB_C-: now also U1.32 (PA11)
- net SCL1: now reaches R12.1, U2.5 (SCL)
- net SCL1: now also U1.42 (PB6)
- net SDA1: now reaches R11.1, U2.4 (SDA)
- net SDA1: now also U1.43 (PB7)
- net 3.3VD: now reaches U1.1 (VBAT)
- net 3.3VD: now also C10.2, C12.1, C13.1, C9.1, R11.2, R12.2, R13.1, U1.24 (VDD), U1.36 (VDD), U1.48 (VDD), U2.6 (VS), U4.2 (VO), C16.1, C17.1, C18.1, C19.1, C20.1, C22.1, FB1.2, J2.1 (Pin_1), R15.1, R25.1, SW3.3 (C), U5.2 (VCC_IN)
- net at U1.20 (PB2): now also R27.2
- net SCL2: now reaches U1.21 (PB10)
- net SCL2: now also U5.3 (SCL)
- net SDA2: now reaches U1.22 (PB11)
- net SDA2: now also U5.4 (SDA)
- net SWDIO: now reaches U1.34 (PA13)
- net SWDIO: now also J2.2 (Pin_2)
- net SWCLK: now reaches U1.37 (PA14)
- net SWCLK: now also J2.3 (Pin_3)
- net at U1.44 (BOOT0): now also R26.2
- net at U1.7 (NRST): now also C15.1, R15.2, SW2.2
- net 3.3VA: now reaches U1.9 (VDDA)
- net 3.3VA: now also R22.2, R7.2, C21.2, C23.2, FB1.1
- net IN+: now reaches U2.10 (Vin+)
- net IN+: now also C14.1, J7.1 (Pin_1), R5.2
- net IN-: now reaches U2.8 (Vbus)
- net IN-: now also U2.9 (Vin-), C14.2, J8.1 (Pin_1), R14.2
- removed net 3.3V: C10.2, C12.1, C13.1, C9.1, R11.2, R12.2, R13.1, R22.2, R7.2, U2.6 (VS), U4.2 (VO)
- new net: R15_Shunt1.2, R5.1
- new net: R14.1, R15_Shunt1.1
- new net: C5.1, R6.2
- new net: R26.1, SW3.2 (B)
- no-connect marks 5 -> 31
Other:
- note added: "Khối Nguồn và Bootloader"
- note added: "Khối hiển thị"
- note added: "Khối vi điều khiển"
- note added: "Khối đo dòng AC"
- note added: "Khối đo dòng, áp, công suất DC"
- note added: "Khối đo áp AC"
- moved on the sheet: C10, C12, C13, C2, C3, C4, C8, C9, D1, D2, D3, D4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

Commit message: update 24/06/2026
Parts:
- removed J2: Conn_01x04_Socket, Connector_PinSocket_1.00mm:PinSocket_1x04_P1.00mm_Vertical, symbol Connector:Conn_01x04_Socket
- added C26: 100nF_Ceramic, Capacitor_THT:C_Disc_D5.0mm_W2.5mm_P2.50mm, symbol PCM_SL_Capacitors:100nF_Ceramic
- added C27: 10uF_16V, Capacitor_THT:CP_Radial_D5.0mm_P2.00mm, symbol PCM_SL_Capacitors:10uF_16V
- added J2: Conn_01x04_Pin, Connector_PinHeader_2.54mm:PinHeader_1x04_P2.54mm_Horizontal, symbol Connector:Conn_01x04_Pin
- added R28: 4.7k, PCM_SparkFun-Resistor:R_0603_1608Metric, symbol PCM_SparkFun-Resistor:4.7k_0603
- added U3: CP2102N-Axx-xQFN28, Package_DFN_QFN:QFN-28-1EP_5x5mm_P0.5mm_EP3.35x3.35mm, symbol Interface_USB:CP2102N-Axx-xQFN28
- FB1: footprint Components_Footprint:XFMR_ZMPT101B -> PCM_Ferrite_SMD_AKL:Ferrite_0805_2012Metric
- J5, J6, J7, J8: footprint Connector:Banana_Jack_1Pin -> (none)
- SW3: footprint Components_Footprint:SOP127P600X165-9N -> (none)
- renumbered R10 to R10_Burden1
Connections:
- net 3.3VD: now also J2.1 (Pin_1)
- net GND: now also C26.1, C27.2, J2.4 (Pin_4), U3.29 (GND), U3.3 (GND)
- net SWCLK: now also J2.3 (Pin_3)
- net SWDIO: now also J2.2 (Pin_2)
- net USB_C+: now also U3.4 (D+)
- net USB_C-: now also U3.5 (D-)
- net VBUS: now also C26.2, C27.1, R28.2, U3.6 (VDD), U3.7 (VREGIN), U3.8 (VBUS)
- net TX: now reaches U1.30 (PA9)
- net TX: now also U3.25 (RXD)
- net RX: now reaches U1.31 (PA10)
- net RX: now also U3.26 (TXD)
- new net: R28.1, U3.9 (~{RST})
- no-connect marks 31 -> 47
Other:
- note added: "Khối Nguồn"
- note removed: "Khối Nguồn và Bootloader"
- moved on the sheet: C8, R10_Burden1, R7, R8

Commit message: update 24/06/2026
Parts:
- J5, J6, J7, J8: footprint (none) -> Components_Footprint:POMONA_73096-2
Changed lines of the file:
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@@
 			)
 		)
-		(property "Footprint" ""
+		(property "Footprint" "Components_Footprint:POMONA_73096-2"
 			(at 78.74 207.01 0)
 			(hide yes)
@@
 			)
 		)
-		(property "Footprint" ""
+		(property "Footprint" "Components_Footprint:POMONA_73096-2"
 			(at 41.91 62.23 0)
 			(hide yes)
@@
 			)
 		)
-		(property "Footprint" ""
+		(property "Footprint" "Components_Footprint:POMONA_73096-2"
 			(at 86.36 62.23 0)
 			(hide yes)
@@
 			)
 		)
-		(property "Footprint" ""
+		(property "Footprint" "Components_Footprint:POMONA_73096-2"
 			(at 34.29 207.01 0)
 			(hide yes)

Commit message: update 26/06/2026
Parts:
- removed U5: DM-OLED096-636, Components_Footprint:MODULE_DM-OLED096-636, symbol DM-OLED096-636:DM-OLED096-636
- added C28, C29, C30, C31, C32: 100nF_Ceramic, Capacitor_THT:C_Disc_D5.0mm_W2.5mm_P2.50mm, symbol PCM_SL_Capacitors:100nF_Ceramic
- added DS1: 4311, Components_Footprint:MODULE_4311, symbol 4311:4311
- added R10, R32, R4: 100, PCM_SparkFun-Resistor:R_0603_1608Metric, symbol PCM_SparkFun-Resistor:100_0603
- added R29, R30, R31, R33, R34: 10k, Resistor_THT:R_Axial_DIN0207_L6.3mm_D2.5mm_P10.16mm_Horizontal, symbol PCM_SL_Resistors:10k
- added SW4: EC11E15244G1, Components_Footprint:EC11E15244G1_AAL, symbol 2026-06-26_06-09-01:EC11E15244G1
- added SW5: Push_Button, Button_Switch_THT:SW_PUSH_6mm, symbol PCM_SL_Devices:Push_Button
- SW3: footprint (none) -> Button_Switch_THT:SW_Slide_SPDT_Straight_CK_OS102011MS2Q
Connections:
- net 3.3VA: now also C32.2
- net 3.3VD: now also DS1.1 (VIN), R29.1, R30.1, R31.1, R33.1
- net GND: now also C28.1, C29.1, C30.1, C31.1, C32.1, DS1.3 (GND), SW4.C, SW4.E, SW5.1
- net TFT_RST: now reaches C15.1, R15.2, SW2.2, U1.7 (NRST)
- net TFT_RST: now also DS1.8 (~{RST})
- net EC_A: now reaches U1.16 (PA6)
- net EC_A: now also R4.1
- net EC_B: now reaches U1.17 (PA7)
- net EC_B: now also R10.1
- net TFT_BLK: now reaches U1.19 (PB1)
- net TFT_BLK: now also DS1.11 (BACKLIGHT)
- net PUSH: now reaches U1.25 (PB12)
- net PUSH: now also R32.2
- net TFT_SCK: now reaches U1.26 (PB13)
- net TFT_SCK: now also DS1.4 (SCK)
- net TFT_MISO: now reaches U1.27 (PB14)
- net TFT_MISO: now also DS1.5 (MISO)
- net TFT_MOSI: now reaches U1.28 (PB15)
- net TFT_MOSI: now also DS1.6 (MOSI)
- net RANGE: now reaches U1.29 (PA8)
- net RANGE: now also R34.2
- net TFT_CS: now reaches U1.45 (PB8)
- net TFT_CS: now also DS1.7 (CS)
- net TFT_DC: now reaches U1.46 (PB9)
- net TFT_DC: now also DS1.9 (D/C)
- new net: C31.2, R33.2, R34.1, SW5.2
- new net: R4.2, SW4.A
- new net: R10.2, SW4.B
- new net: C30.2, R31.2, R32.1, SW4.D
- new net: C29.2, R29.2
- new net: C28.2, R30.2
- no-connect marks 47 -> 39
Other:
- note added: "Khối Bootloader"
- note added: "Khối chọn chế độ"
- moved on the sheet: C11, C15, C16, C17, C18, C19, C20, C26, C27, D7, J2, J5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

Commit message: update 26/06/2026
Parts:
- added J9: 3.5mm, PCM_SparkFun-Connector:ScrewTerminal_1x02_P3.5mm_Horizontal_Black, symbol PCM_SparkFun-Connector:ScrewTerminal_1x02_P3.5mm_Horizontal_Black
Connections:
- net BAT: now also J9.1 (Pin_1)
- net GND: now also J9.2 (Pin_2)
Changed lines of the file:
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@@
 	(wire
 		(pts
+			(xy 394.97 82.55) (xy 397.51 82.55)
+		)
+		(stroke
+			(width 0)
+			(type default)
+		)
+	)
+	(wire
+		(pts
 			(xy 58.42 186.69) (xy 57.15 186.69)
 		)
@@
 	(wire
 		(pts
+			(xy 397.51 85.09) (xy 397.51 86.36)
+		)
+		(stroke
+			(width 0)
+			(type default)
+		)
+	)
+	(wire
+		(pts
 			(xy 182.88 241.3) (xy 193.04 241.3)
 		)
@@
 	(wire
 		(pts
+			(xy 394.97 85.09) (xy 397.51 85.09)
+		)
+		(stroke
+			(width 0)
+			(type default)
+		)
+	)
+	(wire
+		(pts
 			(xy 267.97 88.9) (xy 276.86 88.9)
 		)
@@
 		)
 	)
+	(label "BAT"
+		(at 397.51 82.55 0)
+		(effects
+			(font
+				(size 1.27 1.27)
+			)
+			(justify left bottom)
+		)
+	)
 	(label "USB_C+"
 		(at 233.68 220.98 0)
@@
 	)
 	(symbol
+		(lib_id "PCM_SparkFun-Connector:ScrewTerminal_1x02_P3.5mm_Horizontal_Black")
+		(at 389.89 83.82 0)
+		(mirror y)
+		(unit 1)
+		(body_style 1)
+		(exclude_from_sim no)
+		(in_bom yes)
+		(on_board yes)
+		(in_pos_files yes)
+		(dnp no)
+		(fields_autoplaced yes)
+		(property "Reference" "J9"
+			(at 389.89 76.2 0)
+			(show_name no)
+			(do_not_autoplace no)
+			(effects
+				(font
+					(size 1.27 1.27)
+				)
+			)
+		)
+		(property "Value" "3.5mm"
+			(at 389.89 78.74 0)
+			(show_name no)
+			(do_not_autoplace no)
+			(effects
+				(font
+					(size 1.27 1.27)
+				)
+			)
+		)
+		(property "Footprint" "PCM_SparkFun-Connector:ScrewTerminal_1x02_P3.5mm_Horizontal_Black"
+			(at 389.89 92.71 0)
+			(hide yes)
+			(show_name no)
+			(do_not_autoplace no)
+			(effects
+				(font
+					(size 1.27 1.27)
+				)
+			)
+		)
+		(property "Datasheet" "https://cdn.sparkfun.com/assets/8/5/e/4/d/ASS_4091_CO.pdf"
+			(at 389.89 95.25 0)
+			(hide yes)
+			(show_name no)
+			(do_not_autoplace no)
+			(effects
+				(font
+					(size 1.27 1.27)
+				)
+			)
+		)
+		(property "Description" "Screw terminal"
+			(at 389.89 97.79 0)
+			(hide yes)
+			(show_name no)
+			(do_not_autoplace no)
+			(effects
+				(font
+					(size 1.27 1.27)
+				)
+			)
+		)
+		(property "PROD_ID" "CONN-08399"
+			(at 389.89 90.17 0)
+			(hide yes)
+			(show_name no)
+			(do_not_autoplace no)
+			(effects
+				(font
+					(size 1.27 1.27)
+				)
+			)
+		)
+		(pin "2"
+		)
+		(pin "1"
+		)
+		(instances
+			(project "Energy_Meter"
+				(path "/f1165764-c0ad-44d1-803d-0af7aad26c11"
+					(reference "J9")
+					(unit 1)
+				)
+			)
+		)
+	)
+	(symbol
 		(lib_id "IP5306:IP5306")
 		(at 349.25 44.45 0)
@@
 					(unit 1)
 				)
+			)
+		)
+	)
+	(symbol
+		(lib_name "GND_3")
+		(lib_id "power:GND")
+		(at 397.51 86.36 0)
+		(unit 1)
+		(body_style 1)
+		(exclude_from_sim no)
+		(in_bom yes)
+		(on_board yes)
+		(in_pos_files yes)
+		(dnp no)
+		(fields_autoplaced yes)
+		(property "Reference" "#PWR057"
+			(at 397.51 92.71 0)
+			(hide yes)
+			(show_name no)
+			(do_not_autoplace no)
+			(effects
+				(font
+					(size 1.27 1.27)
+				)
+			)
+		)
+		(property "Value" "GND"
+			(at 397.51 91.44 0)
+			(show_name no)
+			(do_not_autoplace no)
+			(effects
+				(font
+					(size 1.27 1.27)
+				)
+			)
+		)
+		(property "Footprint" ""
+			(at 397.51 86.36 0)
+			(hide yes)
+			(show_name no)
+			(do_not_autoplace no)
+			(effects
+				(font
+					(size 1.27 1.27)
+				)
+			)
+		)
+		(property "Datasheet" ""
+			(at 397.51 86.36 0)
+			(hide yes)
+			(show_name no)
+			(do_not_autoplace no)
+			(effects
+				(font
+					(size 1.27 1.27)
+				)
+			)
+		)
+		(property "Description" "Power symbol creates a global label with name \"GND\" , ground"
+			(at 397.51 86.36 0)
+			(hide yes)
+			(show_name no)
+			(do_not_autoplace no)
+			(effects
+				(font
+					(size 1.27 1.27)
+				)
+			)
+		)
+		(pin "1"
+		)
+		(instances
+			(project "Energy_Meter"
+				(path "/f1165764-c0ad-44d1-803d-0af7aad26c11"
+					(reference "#PWR057")
+					(unit 1)
+				)

Commit message: update 26/06/2026
Parts:
- DS1: MANUFACTURER Adafruit -> (none); Manufacturer (none) -> Adafruit
Changed lines of the file:
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@@
 			)
 		)
-		(property "MANUFACTURER" "Adafruit"
+		(property "Manufacturer" "Adafruit"
 			(at 58.42 254 0)
 			(hide yes)

Commit message: update 30/06/2026
Parts:
- removed C27: 10uF_16V, Capacitor_THT:CP_Radial_D5.0mm_P2.00mm, symbol PCM_SL_Capacitors:10uF_16V
- removed R28: 4.7k, PCM_SparkFun-Resistor:R_0603_1608Metric, symbol PCM_SparkFun-Resistor:4.7k_0603
- removed R34: 10k, Resistor_THT:R_Axial_DIN0207_L6.3mm_D2.5mm_P10.16mm_Horizontal, symbol PCM_SL_Resistors:10k
- removed U3: CP2102N-Axx-xQFN28, Package_DFN_QFN:QFN-28-1EP_5x5mm_P0.5mm_EP3.35x3.35mm, symbol Interface_USB:CP2102N-Axx-xQFN28
- added C33, C35: 22pF, Components_Footprint:CAPRB250W50L400T250H550, symbol FG18C0G1H220JNT00:FG18C0G1H220JNT00
- added R34: 100, PCM_SparkFun-Resistor:R_0603_1608Metric, symbol PCM_SparkFun-Resistor:100_0603
- added TP1, TP10, TP11, TP12, TP13, TP14, TP15, TP16, TP17, TP18, TP19, TP2, TP20, TP21, TP3, TP4, TP5, TP6, TP7, TP8, TP9: 0.5mm, PCM_SparkFun-Connector:TestPoint-0.5mm, symbol PCM_SparkFun-Connector:TestPoint_0.5mm
- added U3: CH340C, Package_SO:SOIC-16_3.9x9.9mm_P1.27mm, symbol Interface_USB:CH340C
- added Y1: Crystal_8MHz, Crystal:Crystal_HC49-4H_Vertical, symbol PCM_SL_Devices:Crystal_8MHz
Connections:
- net 3.3VA: now also TP15.1
- net 3.3VD: now also C26.2, TP11.1, TP14.1, U3.16 (VCC), U3.4 (V3)
- net 5V: now also TP16.1
- net ADC1: now also TP4.1
- net ADC2: now also TP1.1
- net BAT: now also TP18.1
- net GND: now also C33.2, C35.2, TP17.1, TP21.1, TP3.1, TP6.1, U3.1 (GND)
- net IN-: now also TP12.1
- net RANGE: now also R34.2
- net RX: now also TP19.1, U3.2 (TXD)
- net SCL1: now also TP10.1
- net SDA1: now also TP9.1
- net TX: now also TP20.1, U3.3 (RXD)
- net USB_C+: now also U3.5 (UD+)
- net USB_C-: now also U3.6 (UD-)
- net VBUS: now also TP13.1; no longer C26.2
- net at C31.2, R33.2, SW5.2: now also R34.1
- net at R15_Shunt1.2, R5.1: now also TP7.1
- net at C11.1, R22.1, R23.2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: now also TP2.1
- net at R14.1, R15_Shunt1.1: now also TP8.1
- net at R4.2, SW4.A: now also C29.2, R29.2
- net at R10.2, SW4.B: now also C28.2, R30.2
- net at C8.1, J1.1, R10_Burden1.2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: now also TP5.1
- net HSE_IN: now reaches U1.5 (PD0)
- net HSE_IN: now also C35.1, Y1.1
- net HSE_OUT: now reaches U1.6 (PD1)
- net HSE_OUT: now also C33.1, Y1.2
- no-connect marks 39 -> 26
Other:
- moved on the sheet: C15, C28, C29, D7, R15, R26, R29, R30, SW2, SW3

Commit message: update 30/06/2026
Parts:
- removed J5, J6, J7, J8: Conn_01x01_Shielded, Components_Footprint:POMONA_73096-2, symbol Connector_Generic_Shielded:Conn_01x01_Shielded
- added J10, J4, J5, J6: Conn_01x01, Components_Footprint:POMONA_73096-2, symbol Connector_Generic:Conn_01x01
Connections:
- net AC_L: now also J4.1 (Pin_1)
- net AC_N: now also J10.1 (Pin_1)
- net IN+: now also J5.1 (Pin_1)
- net IN-: now also J6.1 (Pin_1)
- no-connect marks 26 -> 22
