File: Energy_Meter.kicad_sch (KiCad schematic)
At the start: 119 parts, among them J1 Conn_Jack_Stereo_3.5mm_SMD_RA, J10 Conn_01x01, J2 Conn_01x04_Pin, J3 USB_C_Receptacle, J4 Conn_01x01, J5 Conn_01x01, J6 Conn_01x01, J9 3.5mm, SW1 SW_Push, SW2 Switch_Tactile_CnK, SW3 SW_SPDT, SW4 EC11E15244G1, SW5 Push_Button, T1 ZMPT101B, U1 STM32F103C8Tx, U2 INA238, U3 CH340C, U4 AMS1117-3.3, U6 IP5306, Y1 Crystal_8MHz

Commit message: update  01/07/2026
Parts:
- removed C1, C2, C3: 10 uF, Capacitor_SMD:C_1206_3216Metric, symbol Device:C
- removed C4, C6, C7: 22 uF, Capacitor_SMD:C_1206_3216Metric, symbol Device:C
- removed C5: 10uF, PCM_SparkFun-Capacitor:C_1210_3225Metric, symbol PCM_SparkFun-Capacitor:10uF_1210_50V_20%
- removed D1, D2, D3, D4: Blue LED, LED_SMD:LED_1206_3216Metric, symbol Device:LED
- removed L1: 1 µH, Inductor_SMD:L_Sunlord_SWPA6028S, symbol Device:L
- removed R3: 2Ω, Resistor_SMD:R_1206_3216Metric, symbol Device:R_US
- removed R6: 2, PCM_fab:R_1206, symbol PCM_fab:R_1206
- removed SW1: SW_Push, Button_Switch_SMD:SW_Tactile_SPST_NO_Straight_CK_PTS636Sx25SMTRLFS, symbol Switch:SW_Push
- removed TP13, TP16, TP18: 0.5mm, PCM_SparkFun-Connector:TestPoint-0.5mm, symbol PCM_SparkFun-Connector:TestPoint_0.5mm
- removed U6: IP5306, Components_Footprint:SOP127P600X165-9N, symbol IP5306:IP5306
- added C27, C34, C39: 10 uF, Capacitor_SMD:C_1206_3216Metric, symbol Device:C
- added C36, C37, C38: 22 uF, Capacitor_SMD:C_1206_3216Metric, symbol Device:C
- added C40: 10uF, PCM_SparkFun-Capacitor:C_1210_3225Metric, symbol PCM_SparkFun-Capacitor:10uF_1210_50V_20%
- added D10, D5, D8, D9: Blue LED, LED_SMD:LED_1206_3216Metric, symbol Device:LED
- added L2: 1 µH, Inductor_SMD:L_Sunlord_SWPA6028S, symbol Device:L
- added R28: 2Ω, Resistor_SMD:R_1206_3216Metric, symbol Device:R_US
- added R35: 2, PCM_fab:R_1206, symbol PCM_fab:R_1206
- added SW6: SW_Push, Button_Switch_SMD:SW_Tactile_SPST_NO_Straight_CK_PTS636Sx25SMTRLFS, symbol Switch:SW_Push
- added TP22, TP23, TP24: 0.5mm, PCM_SparkFun-Connector:TestPoint-0.5mm, symbol PCM_SparkFun-Connector:TestPoint_0.5mm
- added U5: IP5306, Components_Footprint:SOP127P600X165-9N, symbol New_Library:IP5306
- C33, C35: MANUFACTURER TDK -> (none); Manufacturer (none) -> TDK
Connections:
- net 5V: now also C36.1, C37.1, C38.1, TP23.1, U5.8 (VOUT)
- net BAT: now also C39.1, L2.2, R35.1, TP24.1, U5.6 (BAT)
- net GND: now also C27.2, C34.2, C36.2, C37.2, C38.2, C39.2, C40.2, SW6.1, U5.9 (POWERPAD)
- net VBUS: now also C34.1, R28.1, TP22.1, U5.1 (VIN)
- new net: C27.1, R28.2
- new net: D10.2 (A), D5.1 (K), D8.2 (A), D9.1 (K), U5.4 (LED3)
- new net: D10.1 (K), D9.2 (A), U5.3 (LED2)
- new net: SW6.2, U5.5 (KEY)
- new net: C40.1, R35.2
- new net: D5.2 (A), D8.1 (K), U5.2 (LED1)
- new net: L2.1, U5.7 (SW)
Other:
- moved on the sheet: C11, D7, J10, J3, J4, R1, R16, R17, R18, R19, R2, R20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

Commit message: update 15/07/2026
Parts:
- removed C12: 0.1uF_0603_16V, PCM_4ms_Capacitor:C_0603, symbol PCM_4ms_Capacitor:0.1uF_0603_16V
- removed C13, C22: 1uF_0603_25V, Capacitor_SMD:C_0603_1608Metric, symbol PCM_4ms_Capacitor:1uF_0603_25V
- removed C14: 0.1uF, PCM_SparkFun-Capacitor:C_0603_1608Metric, symbol PCM_SparkFun-Capacitor:0.1uF_0603_100V_10%
- removed C15, C16, C17, C18, C19: 100nF_0603_16V, Capacitor_SMD:C_0603_1608Metric, symbol PCM_4ms_Capacitor:100nF_0603_16V
- removed C20, C21: 10nF_0603_25V, Capacitor_SMD:C_0603_1608Metric, symbol PCM_4ms_Capacitor:10nF_0603_25V
- removed C27, C34, C39: 10 uF, Capacitor_SMD:C_1206_3216Metric, symbol Device:C
- removed C36, C37, C38: 22 uF, Capacitor_SMD:C_1206_3216Metric, symbol Device:C
- removed C40: 10uF, PCM_SparkFun-Capacitor:C_1210_3225Metric, symbol PCM_SparkFun-Capacitor:10uF_1210_50V_20%
- removed D10, D5, D8, D9: Blue LED, LED_SMD:LED_1206_3216Metric, symbol Device:LED
- removed D6, D7: ESD5Z3V3, PCM_Diode_SMD_AKL:D_SOD-523, symbol PCM_Diode_TVS_AKL:ESD5Z3V3
- removed L2: 1 µH, Inductor_SMD:L_Sunlord_SWPA6028S, symbol Device:L
- removed R10, R32, R34, R4: 100, PCM_SparkFun-Resistor:R_0603_1608Metric, symbol PCM_SparkFun-Resistor:100_0603
- removed R10_Burden1: 33_0805, Components_Footprint:RESC2012X60N, symbol RS73G2ATTD33R0B:RS73G2ATTD33R0B
- removed R11, R12, R13: 4.7k, PCM_SparkFun-Resistor:R_0603_1608Metric, symbol PCM_SparkFun-Resistor:4.7k_0603
- removed R14, R5: 10, PCM_SparkFun-Resistor:R_1206_3216Metric, symbol PCM_SparkFun-Resistor:10_1206
- removed R16, R17, R18, R19, R20, R21: 20k_1206, Components_Footprint:RES_ERA8ARB203V, symbol ERA8ARB203V:ERA8ARB203V
- removed R25: 1.5k_0603, Capacitor_SMD:C_0603_1608Metric, symbol PCM_4ms_Resistor:1.5k_0603
- removed R28: 2Ω, Resistor_SMD:R_1206_3216Metric, symbol Device:R_US
- removed R4_Burden1: 360_1206, Components_Footprint:RESC3116X65N, symbol RC1206FR-07360RL:RC1206FR-07360RL
- removed SW2: Switch_Tactile_CnK, PCM_fab:Button_CnK_PTS636.0_6x3.5mm, symbol PCM_fab:Switch_Tactile_CnK
- removed SW5: Push_Button, Button_Switch_THT:SW_PUSH_6mm, symbol PCM_SL_Devices:Push_Button
- removed U2: INA238, Package_SO:TSSOP-10_3x3mm_P0.5mm, symbol Sensor_Energy:INA238
- removed U3: CH340C, Package_SO:SOIC-16_3.9x9.9mm_P1.27mm, symbol Interface_USB:CH340C
- added C1, C20, C27, C4, C5, C6: 100nF, Capacitor_THT:C_Disc_D5.0mm_W2.5mm_P2.50mm, symbol PCM_SL_Capacitors:100nF_Ceramic
- added C12, C15: 1uF_50V, Capacitor_THT:CP_Radial_D4.0mm_P1.50mm, symbol PCM_SL_Capacitors:1uF_50V
- added C14, C21, C22: 22uF, Capacitor_THT:CP_Radial_D5.0mm_P2.00mm, symbol PCM_SL_Capacitors:22uF_25V
- added C16: 10nF, Capacitor_THT:C_Disc_D5.0mm_W2.5mm_P2.50mm, symbol PCM_SL_Capacitors:10nF_Ceramic
- added C17, C18, C19: 10uF_16V, Capacitor_THT:CP_Radial_D5.0mm_P2.00mm, symbol PCM_SL_Capacitors:10uF_16V
- added C2: 10uF_63V, Capacitor_THT:CP_Radial_D5.0mm_P2.00mm, symbol PCM_SL_Capacitors:10uF_63V
- added C3: 10nF_Ceramic, Capacitor_THT:C_Disc_D5.0mm_W2.5mm_P2.50mm, symbol PCM_SL_Capacitors:10nF_Ceramic
- added C7: 100nF_Ceramic, Capacitor_THT:C_Disc_D5.0mm_W2.5mm_P2.50mm, symbol PCM_SL_Capacitors:100nF_Ceramic
- added D1, D2, D3, D4: LED, LED_THT:LED_D3.0mm, symbol PCM_SL_Devices:LED_3mm
- added DZ1, DZ2: 1N4728A, PCM_Diode_THT_AKL:D_DO-41_SOD81_P10.16mm_Horizontal_Zener, symbol PCM_Diode_Zener_AKL:1N4728A
- added L1: 1.0uH, PCM_SparkFun-Coil:0805, symbol PCM_SparkFun-Coil:1.0uH_0805_1.45A
- added R10, R3, R4, R6: 100ohm, Resistor_THT:R_Axial_DIN0207_L6.3mm_D2.5mm_P10.16mm_Horizontal, symbol PCM_SL_Resistors:100ohm
- added R11, R12, R13, R39, R40, R41: 20k, Resistor_THT:R_Axial_DIN0207_L6.3mm_D2.5mm_P10.16mm_Horizontal, symbol PCM_SL_Resistors:20k
- added R14, R5: 10R_0.5W, Resistor_THT:R_Axial_DIN0309_L9.0mm_D3.2mm_P15.24mm_Horizontal, symbol PCM_SL_Devices:Resistor_0.5W
- added R25: 360R_1W, Resistor_THT:R_Axial_DIN0414_L11.9mm_D4.5mm_P20.32mm_Horizontal, symbol PCM_SL_Devices:Resistor_1W
- added R28, R37, R38: 4.7k, Resistor_THT:R_Axial_DIN0207_L6.3mm_D2.5mm_P10.16mm_Horizontal, symbol PCM_SL_Resistors:4.7k
- added R32: 33R_1%_2512, PCM_Resistor_SMD_AKL:R_2512_6332Metric, symbol PCM_Resistor_AKL:R_2512
- added R34: 1.5k, Resistor_THT:R_Axial_DIN0207_L6.3mm_D2.5mm_P10.16mm_Horizontal, symbol PCM_SL_Resistors:1.5k
- added R36: 2, PCM_fab:R_1206, symbol PCM_fab:R_1206
- added SW7, SW8: SW_Push, Button_Switch_SMD:SW_Tactile_SPST_NO_Straight_CK_PTS636Sx25SMTRLFS, symbol Switch:SW_Push
- added TP13, TP16: 0.5mm, PCM_SparkFun-Connector:TestPoint-0.5mm, symbol PCM_SparkFun-Connector:TestPoint_0.5mm
- added U3: CH340G, Package_SO:SOIC-16_3.9x9.9mm_P1.27mm, symbol Interface_USB:CH340G
- added U6: INA226, Package_SO:TSSOP-10_3x3mm_P0.5mm, symbol Sensor_Energy:INA226
- C23: value 100nF_Ceramic -> 100nF
- J10, J4, J5, J6: footprint Components_Footprint:POMONA_73096-2 -> MountingHole:MountingHole_4.3mm_M4_Pad_Via
- R1, R2: Part Number (none) -> ERJ-8GEYJ512V
- SW6: Part Number (none) -> PTS636 SK25 SMTR LFS
- U1: Part Number (none) -> STM32F103C8T6TR
- U4: Part Number (none) -> AMS1117-3.3
- U5: MANUFACTURER Injoinic -> (none); Manufacturer (none) -> Injoinic
Connections:
- net 3.3VA: now also C16.2
- net 3.3VD: now also C1.2, C12.1, C15.1, C27.2, C3.2, C4.2, C5.2, C6.2, R28.2, R34.2, R37.2, R38.1, U3.16 (VCC), U3.4 (V3), U6.6 (VS)
- net 5V: now also C14.1, C21.1, C22.1
- net AC_L: now also R11.1
- net AC_N: now also R39.2
- net ADC1: now also DZ1.1 (K)
- net ADC2: now also DZ2.1 (K)
- net BAT: now also C19.1, L1.2
- net EC_A: now also R3.1
- net EC_B: now also R4.2
- net GND: now also C1.1, C12.2, C14.2, C15.2, C16.1, C17.2, C18.2, C19.2, C2.2, C21.2, C22.2, C27.1, C3.1, C4.1, C5.1, C6.1, C7.1, DZ1.2 (A), DZ2.2 (A), SW7.1, SW8.1, U3.1 (GND), U6.1 (A1), U6.2 (A0), U6.7 (GND)
- net IN+: now also C20.2, R5.2, U6.10 (Vin+)
- net IN-: now also C20.1, R14.1, U6.8 (Vbus), U6.9 (Vin-)
- net PUSH: now also R6.2
- net RANGE: now also R10.2
- net RX: now also U3.2 (TXD)
- net SCL1: now also R37.1, U6.5 (SCL)
- net SDA1: now also R28.1, U6.4 (SDA)
- net TFT_RST: now also C7.2, SW8.2
- net TX: now also U3.3 (RXD)
- net USB_C+: now also R34.1, U3.5 (UD+)
- net USB_C-: now also U3.6 (UD-)
- net VBUS: now also C18.1, R36.1
- net at U5.4 (LED3): now also D1.2, D2.1, D3.2, D4.1
- net at U5.3 (LED2): now also D1.1, D2.2
- net at C31.2, R33.2: now also R10.1, SW7.2
- net at R15_Shunt1.2, TP7.1: now also R5.1
- net at C11.1, R22.1, R23.2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: now also R25.1
- net at J1.2, R9.1: now also R32.2
- net at R15_Shunt1.1, TP8.1: now also R14.2
- net at C29.2, R29.2, SW4.A: now also R3.2
- net at C28.2, R30.2, SW4.B: now also R4.1
- net at C30.2, R31.2, SW4.D: now also R6.1
- net at T1.2: now also R41.2, TP16.1
- net at C8.1, J1.1, R7.1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: now also R32.1
- net at R35.2: now also C2.1
- net at T1.1: now also R13.2, TP13.1
- net at R24.1, T1.3: now also R25.2
- net at U5.2 (LED1): now also D3.1, D4.2
- net at U5.7 (SW): now also L1.1
- new net: R39.1, R40.1
- new net: R38.2, U6.3 (~{Alert})
- new net: C17.1, R36.2
- new net: R40.2, R41.1
- new net: R11.2, R12.1
- new net: R12.2, R13.1
Other:
- moved on the sheet: J10, J4, TP22

Commit message: update 16/07/2026
Parts:
- removed C1, C20, C23, C27, C4, C5, C6: 100nF, Capacitor_THT:C_Disc_D5.0mm_W2.5mm_P2.50mm, symbol PCM_SL_Capacitors:100nF_Ceramic
- removed C10, C25, C26, C28, C29, C30, C31, C32, C7: 100nF_Ceramic, Capacitor_THT:C_Disc_D5.0mm_W2.5mm_P2.50mm, symbol PCM_SL_Capacitors:100nF_Ceramic
- removed C11, C17, C18, C19, C24, C8, C9: 10uF_16V, Capacitor_THT:CP_Radial_D5.0mm_P2.00mm, symbol PCM_SL_Capacitors:10uF_16V
- removed C12, C15: 1uF_50V, Capacitor_THT:CP_Radial_D4.0mm_P1.50mm, symbol PCM_SL_Capacitors:1uF_50V
- removed C14, C21, C22: 22uF, Capacitor_THT:CP_Radial_D5.0mm_P2.00mm, symbol PCM_SL_Capacitors:22uF_25V
- removed C16: 10nF, Capacitor_THT:C_Disc_D5.0mm_W2.5mm_P2.50mm, symbol PCM_SL_Capacitors:10nF_Ceramic
- removed C2: 10uF_63V, Capacitor_THT:CP_Radial_D5.0mm_P2.00mm, symbol PCM_SL_Capacitors:10uF_63V
- removed C3: 10nF_Ceramic, Capacitor_THT:C_Disc_D5.0mm_W2.5mm_P2.50mm, symbol PCM_SL_Capacitors:10nF_Ceramic
- removed D1, D2, D3, D4: LED, LED_THT:LED_D3.0mm, symbol PCM_SL_Devices:LED_3mm
- removed R10, R3, R4, R6: 100ohm, Resistor_THT:R_Axial_DIN0207_L6.3mm_D2.5mm_P10.16mm_Horizontal, symbol PCM_SL_Resistors:100ohm
- removed R11, R12, R13, R39, R40, R41: 20k, Resistor_THT:R_Axial_DIN0207_L6.3mm_D2.5mm_P10.16mm_Horizontal, symbol PCM_SL_Resistors:20k
- removed R15, R26, R27, R29, R30, R31, R33: 10k, Resistor_THT:R_Axial_DIN0207_L6.3mm_D2.5mm_P10.16mm_Horizontal, symbol PCM_SL_Resistors:10k
- removed R22, R23, R7, R8: 470k, Resistor_THT:R_Axial_DIN0207_L6.3mm_D2.5mm_P10.16mm_Horizontal, symbol PCM_SL_Resistors:470k
- removed R24, R9: 1k, Resistor_THT:R_Axial_DIN0207_L6.3mm_D2.5mm_P10.16mm_Horizontal, symbol PCM_SL_Resistors:1k
- removed R25: 360R_1W, Resistor_THT:R_Axial_DIN0414_L11.9mm_D4.5mm_P20.32mm_Horizontal, symbol PCM_SL_Devices:Resistor_1W
- removed R28, R37, R38: 4.7k, Resistor_THT:R_Axial_DIN0207_L6.3mm_D2.5mm_P10.16mm_Horizontal, symbol PCM_SL_Resistors:4.7k
- added C1, C2: 1uF_1206, Components_Footprint:CAPC3216X180N, symbol CL31B105KCHNNNE:CL31B105KCHNNNE
- added C10, C17, C18, C19, C23, C24, C25, C26, C42, C43, C45, C46, C47, C48, C9: 100nF_1206_10%, Components_Footprint:CAPC3216X100N, symbol CL31B104KBCNNNC:CL31B104KBCNNNC
- added C13, C34, C36, C37, C38, C39, C40, C41: 10uF, PCM_SparkFun-Capacitor:C_0805_2012Metric, symbol PCM_SparkFun-Capacitor:10uF_0805_25V_10%
- added C3, C6, C7: 22uF, PCM_SparkFun-Capacitor:C_1206_3216Metric, symbol PCM_SparkFun-Capacitor:22uF_1206_50V_10%
- added C4, C5: 10nF_1206, Components_Footprint:CAPC3216X90N, symbol VJ1206Y103KXACW1BC:VJ1206Y103KXACW1BC
- added C44: 100nF_1206, Components_Footprint:CAPC3216X100N, symbol CL31B104KBCNNNC:CL31B104KBCNNNC
- added D5, D6, D7, D8: Blue, PCM_SparkFun-LED:LED_1206_3216Metric_Blue, symbol PCM_SparkFun-LED:LED_Blue_1206
- added R11, R12, R13, R15, R26, R29: 20k_1206_1%, Components_Footprint:RESC3216X70N, symbol RN73R2BTTD2002F25:RN73R2BTTD2002F25
- added R16, R17, R18: 4.7k_0805, Components_Footprint:RESC2012X60N, symbol RNCP0805FTD4K75:RNCP0805FTD4K75
- added R19, R20, R21, R28, R37, R38, R42: 10k_1206, PCM_fab:R_1206, symbol PCM_fab:R_1206
- added R22, R23, R24, R25: 100R_1206, PCM_fab:R_1206, symbol PCM_fab:R_1206
- added R27, R30, R31, R33: 470k_1206, PCM_fab:R_1206, symbol PCM_fab:R_1206
- added R7, R8: 1k_2512, PCM_Resistor_SMD_AKL:R_2512_6332Metric, symbol PCM_Resistor_AKL:R_2512
- added R9: 360_1206, Components_Footprint:RESC3116X65N, symbol Energy_Meter_Sym_Lib:RC1206FR-07360RL
Connections:
- net 3.3VA: now also C17.1, C48.1, C5.1, R27.1, R31.1
- net 3.3VD: now also C1.1, C2.1, C25.1, C26.1, C38.1, C4.1, C43.1, C44.1, C45.1, C46.1, C9.1, R16.2, R17.2, R18.1, R19.1, R28.1, R37.1, R38.1, R42.1
- net 5V: now also C10.1, C3.1, C39.1, C6.1, C7.1
- net AC_L: now also R11.1
- net AC_N: now also R12.1
- net ADC1: now also R7.1
- net ADC2: now also R8.2
- net BAT: now also C37.1
- net EC_A: now also R22.1
- net EC_B: now also R23.2
- net GND: now also C1.2, C10.2, C13.2, C17.2, C18.2, C19.2, C2.2, C23.2, C24.2, C25.2, C26.2, C3.2, C34.2, C36.2, C37.2, C38.2, C39.2, C4.2, C40.2, C41.2, C43.2, C44.2, C45.2, C46.2, C47.2, C48.2, C5.2, C6.2, C7.2, C9.2, R20.1, R30.2, R33.1
- net IN+: now also C42.1
- net IN-: now also C42.2
- net PUSH: now also R24.2
- net RANGE: now also R25.2
- net SCL1: now also R16.1
- net SDA1: now also R17.1
- net TFT_RST: now also C47.1, R19.2
- net VBUS: now also C34.1
- net at SW7.2: now also C18.1, R25.1, R42.2
- net at T1.4, TP2.1: now also C41.1, R31.2, R33.2, R9.1
- net at J1.2, R32.2: now also R7.2
- net at SW4.A: now also C23.1, R22.2, R28.2
- net at SW4.B: now also C24.1, R23.1, R37.2
- net at SW4.D: now also C19.1, R24.1, R38.2
- net at T1.3: now also R8.1, R9.2
- net at U6.3 (~{Alert}): now also R18.2
- net at U5.4 (LED3): now also D5.2 (A), D6.1 (K), D7.2 (A), D8.1 (K)
- net at U5.2 (LED1): now also D7.1 (K), D8.2 (A)
- net at R36.2: now also C13.1
- net at U1.20 (PB2): now also R20.2
- net at T1.2, TP16.1: now also R29.2
- net at R35.2: now also C36.1
- net at J1.1, R32.1, TP5.1: now also C40.1, R27.2, R30.1
- net at SW3.2 (B): now also R21.1
- net at T1.1, TP13.1: now also R26.2
- net at U5.3 (LED2): now also D5.1 (K), D6.2 (A)
- net at U1.44 (BOOT0): now also R21.2
- new net: R12.2, R13.1
- new net: R13.2, R29.1
- new net: R11.2, R15.1
- new net: R15.2, R26.1
Other:
- moved on the sheet: R15_Shunt1, R32, SW3, SW8, TP15, TP21

Commit message: update 16/07/2026
Connections:
- net EC_A: now also U1.17 (PA7); no longer U1.16 (PA6)
- net EC_B: now also U1.16 (PA6); no longer U1.17 (PA7)
- net SCL2: no longer names the net of U1.21 (PB10)
- net SDA2: no longer names the net of U1.22 (PB11)
- no-connect marks 22 -> 24
Changed lines of the file:
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@@
 	)
 	(no_connect
+		(at 193.04 243.84)
+	)
+	(no_connect
 		(at 364.49 168.91)
 	)
@@
 	)
 	(no_connect
+		(at 193.04 246.38)
+	)
+	(no_connect
 		(at 193.04 228.6)
 	)
@@
 	(wire
 		(pts
-			(xy 182.88 243.84) (xy 193.04 243.84)
-		)
-		(stroke
-			(width 0)
-			(type default)
-		)
-	)
-	(wire
-		(pts
 			(xy 58.42 173.99) (xy 57.15 173.99)
 		)
@@
 	(wire
 		(pts
-			(xy 182.88 246.38) (xy 193.04 246.38)
-		)
-		(stroke
-			(width 0)
-			(type default)
-		)
-	)
-	(wire
-		(pts
 			(xy 158.75 181.61) (xy 158.75 182.88)
 		)
@@
 		)
 	)
-	(label "SDA2"
-		(at 182.88 246.38 0)
-		(effects
-			(font
-				(size 1.27 1.27)
-			)
-			(justify left bottom)
-		)
-	)
 	(label "TFT_CS"
 		(at 182.88 238.76 0)
@@
 	)
 	(label "EC_B"
-		(at 233.68 208.28 0)
+		(at 233.68 205.74 0)
 		(effects
 			(font
@@
 		)
 	)
-	(label "SCL2"
-		(at 182.88 243.84 0)
-		(effects
-			(font
-				(size 1.27 1.27)
-			)
-			(justify left bottom)
-		)
-	)
 	(label "TFT_SCK"
 		(at 182.88 251.46 0)
@@
 	)
 	(label "EC_A"
-		(at 233.68 205.74 0)
+		(at 233.68 208.28 0)
 		(effects
 			(font

Commit message: update 17/07/2026
Parts:
- removed C1, C2: 1uF_1206, Components_Footprint:CAPC3216X180N, symbol CL31B105KCHNNNE:CL31B105KCHNNNE
- removed C10, C17, C18, C19, C23, C24, C25, C26, C42, C43, C45, C46, C47, C48, C9: 100nF_1206_10%, Components_Footprint:CAPC3216X100N, symbol CL31B104KBCNNNC:CL31B104KBCNNNC
- removed C3, C6, C7: 22uF, PCM_SparkFun-Capacitor:C_1206_3216Metric, symbol PCM_SparkFun-Capacitor:22uF_1206_50V_10%
- removed C33, C35: 22pF, Components_Footprint:CAPRB250W50L400T250H550, symbol FG18C0G1H220JNT00:FG18C0G1H220JNT00
- removed C4, C5: 10nF_1206, Components_Footprint:CAPC3216X90N, symbol VJ1206Y103KXACW1BC:VJ1206Y103KXACW1BC
- removed C40: 10uF, PCM_SparkFun-Capacitor:C_0805_2012Metric, symbol PCM_SparkFun-Capacitor:10uF_0805_25V_10%
- removed C44: 100nF_1206, Components_Footprint:CAPC3216X100N, symbol CL31B104KBCNNNC:CL31B104KBCNNNC
- removed D5, D6, D7, D8: Blue, PCM_SparkFun-LED:LED_1206_3216Metric_Blue, symbol PCM_SparkFun-LED:LED_Blue_1206
- removed DZ1, DZ2: 1N4728A, PCM_Diode_THT_AKL:D_DO-41_SOD81_P10.16mm_Horizontal_Zener, symbol PCM_Diode_Zener_AKL:1N4728A
- removed R14, R5: 10R_0.5W, Resistor_THT:R_Axial_DIN0309_L9.0mm_D3.2mm_P15.24mm_Horizontal, symbol PCM_SL_Devices:Resistor_0.5W
- removed R34: 1.5k, Resistor_THT:R_Axial_DIN0207_L6.3mm_D2.5mm_P10.16mm_Horizontal, symbol PCM_SL_Resistors:1.5k
- removed SW3: SW_SPDT, Button_Switch_THT:SW_Slide_SPDT_Straight_CK_OS102011MS2Q, symbol Switch:SW_SPDT
- removed Y1: Crystal_8MHz, Crystal:Crystal_HC49-4H_Vertical, symbol PCM_SL_Devices:Crystal_8MHz
- added C1, C2: 22pF_0805, Components_Footprint:CAPC2012X88N, symbol C0805C220K5GACTU:C0805C220K5GACTU
- added C10, C11, C12, C14, C16, C18, C19, C20, C21, C22, C23, C24, C25, C26, C27, C8: 100nF_0805, PCM_Capacitor_SMD_AKL:C_0805_2012Metric, symbol PCM_Capacitor_AKL:C_0805
- added C15, C17: 10nF_0805, PCM_Capacitor_SMD_AKL:C_0805_2012Metric, symbol PCM_Capacitor_AKL:C_0805
- added C3, C6: 1.0uF, PCM_SparkFun-Capacitor:C_0805_2012Metric, symbol PCM_SparkFun-Capacitor:1.0uF_0805_25V_10%
- added C4, C5, C9: 22uF, PCM_SparkFun-Capacitor:C_0805_2012Metric, symbol PCM_SparkFun-Capacitor:22uF_0805_25V_20%
- added C43: 10uF, PCM_SparkFun-Capacitor:C_0805_2012Metric, symbol PCM_SparkFun-Capacitor:10uF_0805_25V_10%
- added D1, D2, D3, D4: Red, PCM_SparkFun-LED:LED_1206_3216Metric_Red, symbol PCM_SparkFun-LED:LED_Red_1206
- added D5, D6: PESD5Z3.3, PCM_Diode_SMD_AKL:D_SOD-523, symbol PCM_Diode_TVS_AKL:PESD5Z3.3
- added R4, R6: 10R_0805, PCM_Resistor_SMD_AKL:R_0805_2012Metric, symbol PCM_Resistor_AKL:R_0805
- added X1: SMD5032-4, PCM_Crystal_AKL:Crystal_SMD_5032-4Pin_5.0x3.2mm, symbol PCM_Crystal_AKL:SMD5032-4
Connections:
- net 3.3VA: now also C16.1, C17.1, C22.1
- net 3.3VD: now also R21.1, C11.1, C12.1, C14.1, C15.1, C21.2, C23.1, C24.1, C3.1, C6.1, C8.1
- net 5V: now also C20.1, C4.1, C5.1, C9.1
- net ADC1: now also D6.1 (K)
- net ADC2: now also D5.1 (K)
- net GND: now also C1.1, C10.2, C11.2, C12.2, C14.2, C15.2, C16.2, C17.2, C18.2, C19.2, C2.2, C20.2, C21.1, C22.2, C23.2, C24.2, C25.2, C27.2, C3.2, C4.2, C43.2, C5.2, C6.2, C8.2, C9.2, D5.2 (A), D6.2 (A), X1.2, X1.4
- net HSE_IN: now also C1.2, X1.1
- net HSE_OUT: now also C2.1, X1.3
- net IN+: now also C26.1, R6.2
- net IN-: now also C26.2, R4.1
- net TFT_RST: now also C25.1
- net USB_C+: no longer U1.33 (PA12)
- net USB_C-: no longer U1.32 (PA11)
- net at R25.1, R42.2, SW7.2: now also C18.1
- net at R15_Shunt1.1, TP8.1: now also R4.2
- net at R15_Shunt1.2, TP7.1: now also R6.1
- net at R22.2, R28.2, SW4.A: now also C10.1
- net at R23.1, R37.2, SW4.B: now also C27.1
- net at R24.1, R38.2, SW4.D: now also C19.1
- net at J1.1, R27.2, R30.1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: now also C43.1
- net at U5.3 (LED2): now also D1.1 (K), D2.2 (A)
- net at U5.4 (LED3): now also D1.2 (A), D2.1 (K), D3.2 (A), D4.1 (K)
- net at U5.2 (LED1): now also D3.1 (K), D4.2 (A)
- no-connect marks 24 -> 26
Other:
- moved on the sheet: R21, R25, R27, R30, R42, SW7, TP19, TP20, TP5, U3

Commit message: update 18/07/2026
Parts:
- removed R20: 10k_1206, PCM_fab:R_1206, symbol PCM_fab:R_1206
- added R3: 10k, PCM_SparkFun-Resistor:R_0603_1608Metric, symbol PCM_SparkFun-Resistor:10k_0603
Connections:
- net GND: now also R3.1
- net at U1.20 (PB2): now also R3.2
Changed lines of the file:
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@@
 	(wire
 		(pts
-			(xy 167.64 223.52) (xy 165.1 223.52)
+			(xy 165.1 223.52) (xy 170.18 223.52)
 		)
 		(stroke
@@
 	(wire
 		(pts
+			(xy 175.26 223.52) (xy 193.04 223.52)
+		)
+		(stroke
+			(width 0)
+			(type default)
+		)
+	)
+	(wire
+		(pts
 			(xy 182.88 233.68) (xy 193.04 233.68)
 		)
@@
 	(wire
 		(pts
-			(xy 177.8 223.52) (xy 193.04 223.52)
-		)
-		(stroke
-			(width 0)
-			(type default)
-		)
-	)
-	(wire
-		(pts
 			(xy 20.32 111.76) (xy 19.05 111.76)
 		)
@@
 	)
 	(symbol
+		(lib_id "PCM_SparkFun-Resistor:10k_0603")
+		(at 172.72 223.52 0)
+		(unit 1)
+		(body_style 1)
+		(exclude_from_sim no)
+		(in_bom yes)
+		(on_board yes)
+		(in_pos_files yes)
+		(dnp no)
+		(fields_autoplaced yes)
+		(property "Reference" "R3"
+			(at 172.72 217.17 0)
+			(show_name no)
+			(do_not_autoplace no)
+			(effects
+				(font
+					(size 1.27 1.27)
+				)
+			)
+		)
+		(property "Value" "10k"
+			(at 172.72 219.71 0)
+			(show_name no)
+			(do_not_autoplace no)
+			(effects
+				(font
+					(size 1.27 1.27)
+				)
+			)
+		)
+		(property "Footprint" "PCM_SparkFun-Resistor:R_0603_1608Metric"
+			(at 172.72 227.838 0)
+			(hide yes)
+			(show_name no)
+			(do_not_autoplace no)
+			(effects
+				(font
+					(size 1.27 1.27)
+				)
+			)
+		)
+		(property "Datasheet" "https://www.vishay.com/docs/20035/dcrcwe3.pdf"
+			(at 172.72 232.41 0)
+			(hide yes)
+			(show_name no)
+			(do_not_autoplace no)
+			(effects
+				(font
+					(size 1.27 1.27)
+				)
+			)
+		)
+		(property "Description" "Resistor"
+			(at 172.72 234.95 0)
+			(hide yes)
+			(show_name no)
+			(do_not_autoplace no)
+			(effects
+				(font
+					(size 1.27 1.27)
+				)
+			)
+		)
+		(property "PROD_ID" "RES-00824"
+			(at 172.72 229.87 0)
+			(hide yes)
+			(show_name no)
+			(do_not_autoplace no)
+			(effects
+				(font
+					(size 1.27 1.27)
+				)
+			)
+		)
+		(pin "2"
+		)
+		(pin "1"
+		)
+		(instances
+			(project "Energy_Meter"
+				(path "/f1165764-c0ad-44d1-803d-0af7aad26c11"
+					(reference "R3")
+					(unit 1)
+				)
+			)
+		)
+	)
+	(symbol
 		(lib_id "PCM_SparkFun-PowerSymbol:3.3V")
 		(at 152.4 87.63 0)
@@
 					(unit 1)
 				)
-			)
-		)
-	)
-	(symbol
-		(lib_id "PCM_fab:R_1206")
-		(at 172.72 223.52 90)
-		(unit 1)
-		(body_style 1)
-		(exclude_from_sim no)
-		(in_bom yes)
-		(on_board yes)
-		(in_pos_files yes)
-		(dnp no)
-		(fields_autoplaced yes)
-		(property "Reference" "R20"
-			(at 172.72 217.17 90)
-			(show_name no)
-			(do_not_autoplace no)
-			(effects
-				(font
-					(size 1.27 1.27)
-				)
-			)
-		)
-		(property "Value" "10k_1206"
-			(at 172.72 219.71 90)
-			(show_name no)
-			(do_not_autoplace no)
-			(effects
-				(font
-					(size 1.27 1.27)
-				)
-			)
-		)
-		(property "Footprint" "PCM_fab:R_1206"
-			(at 172.72 223.52 90)
-			(hide yes)
-			(show_name no)
-			(do_not_autoplace no)
-			(effects
-				(font
-					(size 1.27 1.27)
-				)
-			)
-		)
-		(property "Datasheet" ""
-			(at 172.72 223.52 0)
-			(hide yes)
-			(show_name no)
-			(do_not_autoplace no)
-			(effects
-				(font
-					(size 1.27 1.27)
-				)
-			)
-		)
-		(property "Description" "Resistor"
-			(at 172.72 223.52 0)
-			(hide yes)
-			(show_name no)
-			(do_not_autoplace no)
-			(effects
-				(font
-					(size 1.27 1.27)
-				)
-			)
-		)
-		(pin "2"
-		)
-		(pin "1"
-		)
-		(instances
-			(project "Energy_Meter"
-				(path "/f1165764-c0ad-44d1-803d-0af7aad26c11"
-					(reference "R20")
-					(unit 1)
-				)
