File: Energy_Meter.kicad_sch (KiCad schematic)
At the start: 119 parts, among them J1 Conn_Jack_Stereo_3.5mm_SMD_RA, J10 Conn_01x01, J2 Conn_01x04_Pin, J3 USB_C_Receptacle, J4 Conn_01x01, J5 Conn_01x01, J6 Conn_01x01, J9 3.5mm, SW4 EC11E15244G1, SW6 SW_Push, SW7 SW_Push, SW8 SW_Push, T1 ZMPT101B, U1 STM32F103C8Tx, U3 CH340G, U4 AMS1117-3.3, U5 IP5306, U6 INA226, X1 SMD5032-4

Commit message: update 20/07/2026
Parts:
- removed R11, R12, R13, R15, R26, R29: 20k_1206_1%, Components_Footprint:RESC3216X70N, symbol RN73R2BTTD2002F25:RN73R2BTTD2002F25
- added R10, R11, R12, R13, R14, R5: 20k_1206, Components_Footprint:RES_ERA8ARB203V, symbol Energy_Meter_Sym_Lib:ERA8ARB203V
- added TP18, TP25, TP26, TP27: 0.5mm, PCM_SparkFun-Connector:TestPoint-0.5mm, symbol PCM_SparkFun-Connector:TestPoint_0.5mm
- J10, J4, J5, J6: footprint MountingHole:MountingHole_4.3mm_M4_Pad_Via -> MountingHole:MountingHole_4.3mm_M4_Pad
Connections:
- net AC_L: now also R5.1
- net AC_N: now also R12.1
- net EC_A: now also TP18.1
- net EC_B: now also TP25.1
- net PUSH: now also TP27.1
- net RANGE: now also TP26.1
- net at T1.1, TP13.1: now also R11.2
- net at T1.2, TP16.1: now also R14.2
- new net: R13.2, R14.1
- new net: R10.2, R11.1
- new net: R12.2, R13.1
- new net: R10.1, R5.2
Other:
- moved on the sheet: C41, D5, J10, J4, R22, R23, R31, R33, R8, R9, T1, TP1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

Commit message: update 22/07/2026
Parts:
- removed C24: 100nF_0805, PCM_Capacitor_SMD_AKL:C_0805_2012Metric, symbol PCM_Capacitor_AKL:C_0805
- removed DS1: 4311, Components_Footprint:MODULE_4311, symbol 4311:4311
- added C28: 100nF_0805, PCM_Capacitor_SMD_AKL:C_0805_2012Metric, symbol PCM_Capacitor_AKL:C_0805
- added DS1: OLED_128X64_1.3_I2C, Components_Footprint:LCD_OLED_128X64_1.3_I2C, symbol OLED_128X64_1.3_I2C:OLED_128X64_1.3_I2C
- added R20, R26: 4.7k_0805, Components_Footprint:RESC2012X60N, symbol RNCP0805FTD4K75:RNCP0805FTD4K75
Connections:
- net 3.3VD: now also C28.1, DS1.1 (VDD), R20.2, R26.2
- net GND: now also C28.2, DS1.2 (GND)
- net SCL2: now reaches U1.21 (PB10)
- net SCL2: now also DS1.3 (SCK), R26.1
- net SDA2: now reaches U1.22 (PB11)
- net SDA2: now also DS1.4 (SDA), R20.1
- net TFT_BLK: no longer names the net of U1.19 (PB1)
- net TFT_CS: no longer names the net of U1.45 (PB8)
- net TFT_DC: no longer names the net of U1.46 (PB9)
- net TFT_MISO: no longer names the net of U1.27 (PB14)
- net TFT_MOSI: no longer names the net of U1.28 (PB15)
- net TFT_SCK: no longer names the net of U1.26 (PB13)
- no-connect marks 26 -> 28
