File: Energy_Meter.kicad_sch (KiCad schematic)
At the start: 125 parts, among them J1 Conn_Jack_Stereo_3.5mm_SMD_RA, J10 Conn_01x01, J2 Conn_01x04_Pin, J3 USB_C_Receptacle, J4 Conn_01x01, J5 Conn_01x01, J6 Conn_01x01, J9 3.5mm, SW4 EC11E15244G1, SW6 SW_Push, SW7 SW_Push, SW8 SW_Push, T1 ZMPT101B, U1 STM32F103C8Tx, U3 CH340G, U4 AMS1117-3.3, U5 IP5306, U6 INA226, X1 SMD5032-4

Commit message: update 29/07/2026
Parts:
- added R15, R29, R34, R39, R46, R47: 0R_0805, PCM_Resistor_SMD_AKL:R_0805_2012Metric, symbol PCM_Resistor_AKL:R_0805
Connections:
- net RX: now also R47.2; no longer U1.31 (PA10)
- net SCL1: now also R15.1; no longer U1.42 (PB6)
- net SCL2: now also R34.1; no longer U1.21 (PB10)
- net SDA1: now also R29.1; no longer U1.43 (PB7)
- net SDA2: now also R39.1; no longer U1.22 (PB11)
- net TX: now also R46.2; no longer U1.30 (PA9)
- new net: R47.1, U1.31 (PA10)
- new net: R46.1, U1.30 (PA9)
- new net: R29.2, U1.43 (PB7)
- new net: R15.2, U1.42 (PB6)
- new net: R34.2, U1.21 (PB10)
- new net: R39.2, U1.22 (PB11)

Commit message: update 29/08/2026
Parts:
- J10, J4, J5, J6: footprint MountingHole:MountingHole_4.3mm_M4_Pad -> MountingHole:MountingHole_4.5mm_Pad
Changed lines of the file:
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@@
 	(text "Khối hiển thị"
 		(exclude_from_sim no)
-		(at 67.31 228.346 0)
+		(at 68.072 219.964 0)
 		(effects
 			(font
@@
 	(text "Khối vi điều khiển"
 		(exclude_from_sim no)
-		(at 209.804 152.654 0)
+		(at 208.534 137.16 0)
 		(effects
 			(font
@@
 			)
 		)
-		(property "Footprint" "MountingHole:MountingHole_4.3mm_M4_Pad"
+		(property "Footprint" "MountingHole:MountingHole_4.5mm_Pad"
 			(at 104.14 63.5 0)
 			(hide yes)
@@
 			)
 		)
-		(property "Footprint" "MountingHole:MountingHole_4.3mm_M4_Pad"
+		(property "Footprint" "MountingHole:MountingHole_4.5mm_Pad"
 			(at 134.62 63.5 0)
 			(hide yes)
@@
 			)
 		)
-		(property "Footprint" "MountingHole:MountingHole_4.3mm_M4_Pad"
+		(property "Footprint" "MountingHole:MountingHole_4.5mm_Pad"
 			(at 34.29 207.01 0)
 			(hide yes)
@@
 			)
 		)
-		(property "Footprint" "MountingHole:MountingHole_4.3mm_M4_Pad"
+		(property "Footprint" "MountingHole:MountingHole_4.5mm_Pad"
 			(at 78.74 207.01 0)
 			(hide yes)
