File: Energy_Meter.kicad_pcb (KiCad board)
At the start: 2 copper layers, 119 parts, among them J1 Conn_Jack_Stereo_3.5mm_SMD_RA, J10 Conn_01x01, J2 Conn_01x04_Pin, J3 USB_C_Receptacle, J4 Conn_01x01, J5 Conn_01x01, J6 Conn_01x01, J9 3.5mm, SW1 SW_Push, SW2 Switch_Tactile_CnK, SW3 SW_SPDT, SW4 EC11E15244G1, SW5 Push_Button, T1 ZMPT101B, U1 STM32F103C8Tx, U2 INA238, U3 CH340C, U4 AMS1117-3.3, U6 IP5306, Y1 Crystal_8MHz

Commit message: update  01/07/2026
Parts:
- removed C1, C2, C3: 10 uF, Capacitor_SMD:C_1206_3216Metric
- removed C10, C23, C25, C26, C28, C29, C30, C31, C32: 100nF_Ceramic, Capacitor_THT:C_Disc_D5.0mm_W2.5mm_P2.50mm
- removed C11, C24, C8, C9: 10uF_16V, Capacitor_THT:CP_Radial_D5.0mm_P2.00mm
- removed C12: 0.1uF_0603_16V, PCM_4ms_Capacitor:C_0603
- removed C13, C22: 1uF_0603_25V, Capacitor_SMD:C_0603_1608Metric
- removed C14: 0.1uF, PCM_SparkFun-Capacitor:C_0603_1608Metric
- removed C15, C16, C17, C18, C19: 100nF_0603_16V, Capacitor_SMD:C_0603_1608Metric
- removed C20, C21: 10nF_0603_25V, Capacitor_SMD:C_0603_1608Metric
- removed C33, C35: 22pF, Components_Footprint:CAPRB250W50L400T250H550
- removed C4, C6, C7: 22 uF, Capacitor_SMD:C_1206_3216Metric
- removed C5: 10uF, PCM_SparkFun-Capacitor:C_1210_3225Metric
- removed D1, D2, D3, D4: Blue LED, LED_SMD:LED_1206_3216Metric
- removed D6, D7: ESD5Z3V3, PCM_Diode_SMD_AKL:D_SOD-523
- removed DS1: 4311, Components_Footprint:MODULE_4311
- removed FB1: FerriteBead, PCM_Ferrite_SMD_AKL:Ferrite_0805_2012Metric
- removed J1: Conn_Jack_Stereo_3.5mm_SMD_RA, PCM_fab:Conn_Jack_Stereo_3.5mm_CUI_SJ-3523-SMT-TR
- removed J10, J4, J5, J6: Conn_01x01, Components_Footprint:POMONA_73096-2
- removed J2: Conn_01x04_Pin, Connector_PinHeader_2.54mm:PinHeader_1x04_P2.54mm_Horizontal
- removed J3: USB_C_Receptacle, PCM_SparkFun-Connector:USB-C_16
- removed J9: 3.5mm, PCM_SparkFun-Connector:ScrewTerminal_1x02_P3.5mm_Horizontal_Black
- removed L1: 1 µH, Inductor_SMD:L_Sunlord_SWPA6028S
- removed R1, R2: 5.1K, Resistor_SMD:R_1206_3216Metric
- removed R10, R32, R34, R4: 100, PCM_SparkFun-Resistor:R_0603_1608Metric
- removed R10_Burden1: 33_0805, Components_Footprint:RESC2012X60N
- removed R11, R12, R13: 4.7k, PCM_SparkFun-Resistor:R_0603_1608Metric
- removed R14, R5: 10, PCM_SparkFun-Resistor:R_1206_3216Metric
- removed R15, R26, R27, R29, R30, R31, R33: 10k, Resistor_THT:R_Axial_DIN0207_L6.3mm_D2.5mm_P10.16mm_Horizontal
- removed R15_Shunt1: 0.001_1%_5W, Components_Footprint:RESC6331X88N
- removed R16, R17, R18, R19, R20, R21: 20k_1206, Components_Footprint:RES_ERA8ARB203V
- removed R22, R23, R7, R8: 470k, Resistor_THT:R_Axial_DIN0207_L6.3mm_D2.5mm_P10.16mm_Horizontal
- removed R24, R9: 1k, Resistor_THT:R_Axial_DIN0207_L6.3mm_D2.5mm_P10.16mm_Horizontal
- removed R25: 1.5k_0603, Capacitor_SMD:C_0603_1608Metric
- removed R3: 2Ω, Resistor_SMD:R_1206_3216Metric
- removed R4_Burden1: 360_1206, Components_Footprint:RESC3116X65N
- removed R6: 2, PCM_fab:R_1206
- removed SW1: SW_Push, Button_Switch_SMD:SW_Tactile_SPST_NO_Straight_CK_PTS636Sx25SMTRLFS
- removed SW2: Switch_Tactile_CnK, PCM_fab:Button_CnK_PTS636.0_6x3.5mm
- removed SW3: SW_SPDT, Button_Switch_THT:SW_Slide_SPDT_Straight_CK_OS102011MS2Q
- removed SW4: EC11E15244G1, Components_Footprint:EC11E15244G1_AAL
- removed SW5: Push_Button, Button_Switch_THT:SW_PUSH_6mm
- removed T1: ZMPT101B, Components_Footprint:XFMR_ZMPT101B
- removed TP1, TP10, TP11, TP12, TP13, TP14, TP15, TP16, TP17, TP18, TP19, TP2, TP20, TP21, TP3, TP4, TP5, TP6, TP7, TP8, TP9: 0.5mm, PCM_SparkFun-Connector:TestPoint-0.5mm
- removed U1: STM32F103C8Tx, Package_QFP:LQFP-48_7x7mm_P0.5mm
- removed U2: INA238, Package_SO:TSSOP-10_3x3mm_P0.5mm
- removed U3: CH340C, Package_SO:SOIC-16_3.9x9.9mm_P1.27mm
- removed U4: AMS1117-3.3, Package_TO_SOT_SMD:SOT-223-3_TabPin2
- removed U6: IP5306, Components_Footprint:SOP127P600X165-9N
- removed Y1: Crystal_8MHz, Crystal:Crystal_HC49-4H_Vertical

Commit message: update 02/07/2026
Parts:
- added C10: 100nF_Ceramic, Capacitor_THT:C_Disc_D5.0mm_W2.5mm_P2.50mm, F.Cu at (183.2, 106.7)
- added C11: 10uF_16V, Capacitor_THT:CP_Radial_D5.0mm_P2.00mm, F.Cu at (126.9, 129.6)
- added C12: 0.1uF_0603_16V, PCM_4ms_Capacitor:C_0603, F.Cu at (214.8, 138.7)
- added C13: 1uF_0603_25V, Capacitor_SMD:C_0603_1608Metric, F.Cu at (189.7, 105.9)
- added C14: 0.1uF, PCM_SparkFun-Capacitor:C_0603_1608Metric, F.Cu at (189.7, 108.4)
- added C15: 100nF_0603_16V, Capacitor_SMD:C_0603_1608Metric, F.Cu at (189.7, 110.9)
- added C16: 100nF_0603_16V, Capacitor_SMD:C_0603_1608Metric, F.Cu at (189.7, 113.4)
- added C17: 100nF_0603_16V, Capacitor_SMD:C_0603_1608Metric, F.Cu at (189.7, 115.9)
- added C18: 100nF_0603_16V, Capacitor_SMD:C_0603_1608Metric, F.Cu at (189.7, 118.5)
- added C19: 100nF_0603_16V, Capacitor_SMD:C_0603_1608Metric, F.Cu at (189.7, 121.0)
- added C20: 10nF_0603_25V, Capacitor_SMD:C_0603_1608Metric, F.Cu at (193.7, 105.9)
- added C21: 10nF_0603_25V, Capacitor_SMD:C_0603_1608Metric, F.Cu at (193.7, 108.4)
- added C22: 1uF_0603_25V, Capacitor_SMD:C_0603_1608Metric, F.Cu at (193.7, 110.9)
- added C23: 100nF_Ceramic, Capacitor_THT:C_Disc_D5.0mm_W2.5mm_P2.50mm, F.Cu at (183.2, 110.7)
- added C24: 10uF_16V, Capacitor_THT:CP_Radial_D5.0mm_P2.00mm, F.Cu at (126.9, 136.2)
- added C25: 100nF_Ceramic, Capacitor_THT:C_Disc_D5.0mm_W2.5mm_P2.50mm, F.Cu at (183.2, 114.8)
- added C26: 100nF_Ceramic, Capacitor_THT:C_Disc_D5.0mm_W2.5mm_P2.50mm, F.Cu at (183.2, 118.8)
- added C27: 10 uF, Capacitor_SMD:C_1206_3216Metric, F.Cu at (196.8, 123.9)
- added C28: 100nF_Ceramic, Capacitor_THT:C_Disc_D5.0mm_W2.5mm_P2.50mm, F.Cu at (183.2, 122.9)
- added C29: 100nF_Ceramic, Capacitor_THT:C_Disc_D5.0mm_W2.5mm_P2.50mm, F.Cu at (183.2, 126.9)
- added C30: 100nF_Ceramic, Capacitor_THT:C_Disc_D5.0mm_W2.5mm_P2.50mm, F.Cu at (183.2, 131.0)
- added C31: 100nF_Ceramic, Capacitor_THT:C_Disc_D5.0mm_W2.5mm_P2.50mm, F.Cu at (183.2, 135.0)
- added C32: 100nF_Ceramic, Capacitor_THT:C_Disc_D5.0mm_W2.5mm_P2.50mm, F.Cu at (183.2, 139.1)
- added C33: 22pF, Components_Footprint:CAPRB250W50L400T250H550, F.Cu at (158.6, 115.3)
- added C34: 10 uF, Capacitor_SMD:C_1206_3216Metric, F.Cu at (196.8, 127.2)
- added C35: 22pF, Components_Footprint:CAPRB250W50L400T250H550, F.Cu at (158.6, 119.3)
- added C36: 22 uF, Capacitor_SMD:C_1206_3216Metric, F.Cu at (196.8, 130.6)
- added C37: 22 uF, Capacitor_SMD:C_1206_3216Metric, F.Cu at (196.8, 133.9)
- added C38: 22 uF, Capacitor_SMD:C_1206_3216Metric, F.Cu at (196.8, 137.3)
- added C39: 10 uF, Capacitor_SMD:C_1206_3216Metric, F.Cu at (196.8, 140.6)
- added C40: 10uF, PCM_SparkFun-Capacitor:C_1210_3225Metric, F.Cu at (164.4, 139.9)
- added C8: 10uF_16V, Capacitor_THT:CP_Radial_D5.0mm_P2.00mm, F.Cu at (126.9, 116.5)
- added C9: 10uF_16V, Capacitor_THT:CP_Radial_D5.0mm_P2.00mm, F.Cu at (126.9, 123.1)
- added D10: Blue LED, LED_SMD:LED_1206_3216Metric, F.Cu at (209.3, 99.9)
- added D5: Blue LED, LED_SMD:LED_1206_3216Metric, F.Cu at (209.3, 89.7)
- added D6: ESD5Z3V3, PCM_Diode_SMD_AKL:D_SOD-523, F.Cu at (202.8, 96.1)
- added D7: ESD5Z3V3, PCM_Diode_SMD_AKL:D_SOD-523, F.Cu at (202.8, 99.4)
- added D8: Blue LED, LED_SMD:LED_1206_3216Metric, F.Cu at (209.3, 93.1)
- added D9: Blue LED, LED_SMD:LED_1206_3216Metric, F.Cu at (209.3, 96.5)
- added DS1: 4311, Components_Footprint:MODULE_4311, F.Cu at (143.1, 82.3)
- added FB1: FerriteBead, PCM_Ferrite_SMD_AKL:Ferrite_0805_2012Metric, F.Cu at (215.2, 132.9)
- added J1: Conn_Jack_Stereo_3.5mm_SMD_RA, PCM_fab:Conn_Jack_Stereo_3.5mm_CUI_SJ-3523-SMT-TR, F.Cu at (210.0, 110.0)
- added J10: Conn_01x01, Components_Footprint:POMONA_73096-2, F.Cu at (171.4, 120.4)
- added J2: Conn_01x04_Pin, Connector_PinHeader_2.54mm:PinHeader_1x04_P2.54mm_Horizontal, F.Cu at (133.4, 115.5)
- added J3: USB_C_Receptacle, PCM_SparkFun-Connector:USB-C_16, F.Cu at (205.0, 123.0)
- added J4: Conn_01x01, Components_Footprint:POMONA_73096-2, F.Cu at (171.4, 61.8)
- added J5: Conn_01x01, Components_Footprint:POMONA_73096-2, F.Cu at (171.4, 81.3)
- added J6: Conn_01x01, Components_Footprint:POMONA_73096-2, F.Cu at (171.4, 100.9)
- added J9: 3.5mm, PCM_SparkFun-Connector:ScrewTerminal_1x02_P3.5mm_Horizontal_Black, F.Cu at (153.0, 129.6)
- added L2: 1 µH, Inductor_SMD:L_Sunlord_SWPA6028S, F.Cu at (165.5, 134.0)
- added R1: 5.1K, Resistor_SMD:R_1206_3216Metric, F.Cu at (214.9, 89.7)
- added R10: 100, PCM_SparkFun-Resistor:R_0603_1608Metric, F.Cu at (193.7, 115.9)
- added R10_Burden1: 33_0805, Components_Footprint:RESC2012X60N, F.Cu at (215.0, 136.0)
- added R11: 4.7k, PCM_SparkFun-Resistor:R_0603_1608Metric, F.Cu at (193.7, 118.5)
- added R12: 4.7k, PCM_SparkFun-Resistor:R_0603_1608Metric, F.Cu at (193.7, 121.0)
- added R13: 4.7k, PCM_SparkFun-Resistor:R_0603_1608Metric, F.Cu at (197.7, 105.9)
- added R14: 10, PCM_SparkFun-Resistor:R_1206_3216Metric, F.Cu at (214.9, 102.9)
- added R15: 10k, Resistor_THT:R_Axial_DIN0207_L6.3mm_D2.5mm_P10.16mm_Horizontal, F.Cu at (182.7, 66.2)
- added R15_Shunt1: 0.001_1%_5W, Components_Footprint:RESC6331X88N, F.Cu at (204.2, 118.5)
- added R16: 20k_1206, Components_Footprint:RES_ERA8ARB203V, F.Cu at (190.8, 123.8)
- added R17: 20k_1206, Components_Footprint:RES_ERA8ARB203V, F.Cu at (190.8, 126.9)
- added R18: 20k_1206, Components_Footprint:RES_ERA8ARB203V, F.Cu at (190.8, 130.1)
- added R19: 20k_1206, Components_Footprint:RES_ERA8ARB203V, F.Cu at (190.8, 133.2)
- added R2: 5.1K, Resistor_SMD:R_1206_3216Metric, F.Cu at (214.9, 93.0)
- added R20: 20k_1206, Components_Footprint:RES_ERA8ARB203V, F.Cu at (190.8, 136.4)
- added R21: 20k_1206, Components_Footprint:RES_ERA8ARB203V, F.Cu at (190.8, 139.5)
- added R22: 470k, Resistor_THT:R_Axial_DIN0207_L6.3mm_D2.5mm_P10.16mm_Horizontal, F.Cu at (182.7, 70.2)
- added R23: 470k, Resistor_THT:R_Axial_DIN0207_L6.3mm_D2.5mm_P10.16mm_Horizontal, F.Cu at (182.7, 74.3)
- added R24: 1k, Resistor_THT:R_Axial_DIN0207_L6.3mm_D2.5mm_P10.16mm_Horizontal, F.Cu at (182.7, 78.3)
- added R25: 1.5k_0603, Capacitor_SMD:C_0603_1608Metric, F.Cu at (197.7, 108.4)
- added R26: 10k, Resistor_THT:R_Axial_DIN0207_L6.3mm_D2.5mm_P10.16mm_Horizontal, F.Cu at (182.7, 82.4)
- added R27: 10k, Resistor_THT:R_Axial_DIN0207_L6.3mm_D2.5mm_P10.16mm_Horizontal, F.Cu at (182.7, 86.4)
- added R28: 2Ω, Resistor_SMD:R_1206_3216Metric, F.Cu at (214.9, 96.3)
- added R29: 10k, Resistor_THT:R_Axial_DIN0207_L6.3mm_D2.5mm_P10.16mm_Horizontal, F.Cu at (182.7, 90.5)
- added R30: 10k, Resistor_THT:R_Axial_DIN0207_L6.3mm_D2.5mm_P10.16mm_Horizontal, F.Cu at (182.7, 94.5)
- added R31: 10k, Resistor_THT:R_Axial_DIN0207_L6.3mm_D2.5mm_P10.16mm_Horizontal, F.Cu at (182.7, 98.6)
- added R32: 100, PCM_SparkFun-Resistor:R_0603_1608Metric, F.Cu at (197.7, 110.9)
- added R33: 10k, Resistor_THT:R_Axial_DIN0207_L6.3mm_D2.5mm_P10.16mm_Horizontal, F.Cu at (182.7, 102.6)
- added R34: 100, PCM_SparkFun-Resistor:R_0603_1608Metric, F.Cu at (197.7, 113.4)
- added R35: 2, PCM_fab:R_1206, F.Cu at (158.7, 123.0)
- added R4: 100, PCM_SparkFun-Resistor:R_0603_1608Metric, F.Cu at (193.7, 113.4)
- added R4_Burden1: 360_1206, Components_Footprint:RESC3116X65N, F.Cu at (203.7, 102.7)
- added R5: 10, PCM_SparkFun-Resistor:R_1206_3216Metric, F.Cu at (214.9, 99.6)
- added R7: 470k, Resistor_THT:R_Axial_DIN0207_L6.3mm_D2.5mm_P10.16mm_Horizontal, F.Cu at (182.7, 54.0)
- added R8: 470k, Resistor_THT:R_Axial_DIN0207_L6.3mm_D2.5mm_P10.16mm_Horizontal, F.Cu at (182.7, 58.1)
- added R9: 1k, Resistor_THT:R_Axial_DIN0207_L6.3mm_D2.5mm_P10.16mm_Horizontal, F.Cu at (182.7, 62.1)
- added SW2: Switch_Tactile_CnK, PCM_fab:Button_CnK_PTS636.0_6x3.5mm, F.Cu at (175.1, 132.7)
- added SW3: SW_SPDT, Button_Switch_THT:SW_Slide_SPDT_Straight_CK_OS102011MS2Q, F.Cu at (198.4, 91.5)
- added SW4: EC11E15244G1, Components_Footprint:EC11E15244G1_AAL, F.Cu at (202.5, 86.4)
- added SW5: Push_Button, Button_Switch_THT:SW_PUSH_6mm, F.Cu at (141.6, 127.5)
- added SW6: SW_Push, Button_Switch_SMD:SW_Tactile_SPST_NO_Straight_CK_PTS636Sx25SMTRLFS, F.Cu at (174.6, 137.9)
- added T1: ZMPT101B, Components_Footprint:XFMR_ZMPT101B, F.Cu at (205.4, 61.1)
- added TP1: 0.5mm, PCM_SparkFun-Connector:TestPoint-0.5mm, F.Cu at (195.3, 95.3)
- added TP10: 0.5mm, PCM_SparkFun-Connector:TestPoint-0.5mm, F.Cu at (196.9, 100.1)
- added TP11: 0.5mm, PCM_SparkFun-Connector:TestPoint-0.5mm, F.Cu at (196.9, 101.7)
- added TP12: 0.5mm, PCM_SparkFun-Connector:TestPoint-0.5mm, F.Cu at (196.9, 103.3)
- added TP14: 0.5mm, PCM_SparkFun-Connector:TestPoint-0.5mm, F.Cu at (198.5, 95.3)
- added TP15: 0.5mm, PCM_SparkFun-Connector:TestPoint-0.5mm, F.Cu at (198.5, 96.9)
- added TP17: 0.5mm, PCM_SparkFun-Connector:TestPoint-0.5mm, F.Cu at (198.5, 98.5)
- added TP19: 0.5mm, PCM_SparkFun-Connector:TestPoint-0.5mm, F.Cu at (198.5, 100.1)
- added TP2: 0.5mm, PCM_SparkFun-Connector:TestPoint-0.5mm, F.Cu at (195.3, 96.9)
- added TP20: 0.5mm, PCM_SparkFun-Connector:TestPoint-0.5mm, F.Cu at (198.5, 101.7)
- added TP21: 0.5mm, PCM_SparkFun-Connector:TestPoint-0.5mm, F.Cu at (198.5, 103.3)
- added TP22: 0.5mm, PCM_SparkFun-Connector:TestPoint-0.5mm, F.Cu at (200.1, 95.3)
- added TP23: 0.5mm, PCM_SparkFun-Connector:TestPoint-0.5mm, F.Cu at (200.1, 96.9)
- added TP24: 0.5mm, PCM_SparkFun-Connector:TestPoint-0.5mm, F.Cu at (200.1, 98.5)
- added TP3: 0.5mm, PCM_SparkFun-Connector:TestPoint-0.5mm, F.Cu at (195.3, 98.5)
- added TP4: 0.5mm, PCM_SparkFun-Connector:TestPoint-0.5mm, F.Cu at (195.3, 100.1)
- added TP5: 0.5mm, PCM_SparkFun-Connector:TestPoint-0.5mm, F.Cu at (195.3, 101.7)
- added TP6: 0.5mm, PCM_SparkFun-Connector:TestPoint-0.5mm, F.Cu at (195.3, 103.3)
- added TP7: 0.5mm, PCM_SparkFun-Connector:TestPoint-0.5mm, F.Cu at (196.9, 95.3)
- added TP8: 0.5mm, PCM_SparkFun-Connector:TestPoint-0.5mm, F.Cu at (196.9, 96.9)
- added TP9: 0.5mm, PCM_SparkFun-Connector:TestPoint-0.5mm, F.Cu at (196.9, 98.5)
- added U1: STM32F103C8Tx, Package_QFP:LQFP-48_7x7mm_P0.5mm, F.Cu at (150.2, 118.9)
- added U2: INA238, Package_SO:TSSOP-10_3x3mm_P0.5mm, F.Cu at (212.3, 118.2)
- added U3: CH340C, Package_SO:SOIC-16_3.9x9.9mm_P1.27mm, F.Cu at (135.4, 131.4)
- added U4: AMS1117-3.3, Package_TO_SOT_SMD:SOT-223-3_TabPin2, F.Cu at (144.5, 138.2)
- added U5: IP5306, Components_Footprint:SOP127P600X165-9N, F.Cu at (155.3, 137.9)
- added Y1: Crystal_8MHz, Crystal:Crystal_HC49-4H_Vertical, F.Cu at (203.7, 134.7)

Commit message: update 15/07/2026
Parts:
- removed C13: 1uF_0603_25V, Capacitor_SMD:C_0603_1608Metric
- removed C34, C39: 10 uF, Capacitor_SMD:C_1206_3216Metric
- removed C36, C37, C38: 22 uF, Capacitor_SMD:C_1206_3216Metric
- removed C40: 10uF, PCM_SparkFun-Capacitor:C_1210_3225Metric
- removed D10, D5, D8, D9: Blue LED, LED_SMD:LED_1206_3216Metric
- removed D6, D7: ESD5Z3V3, PCM_Diode_SMD_AKL:D_SOD-523
- removed L2: 1 µH, Inductor_SMD:L_Sunlord_SWPA6028S
- removed R10_Burden1: 33_0805, Components_Footprint:RESC2012X60N
- removed R16, R17, R18, R19, R20, R21: 20k_1206, Components_Footprint:RES_ERA8ARB203V
- removed R4_Burden1: 360_1206, Components_Footprint:RESC3116X65N
- removed SW2: Switch_Tactile_CnK, PCM_fab:Button_CnK_PTS636.0_6x3.5mm
- removed SW5: Push_Button, Button_Switch_THT:SW_PUSH_6mm
- removed U2: INA238, Package_SO:TSSOP-10_3x3mm_P0.5mm
- added C1: 100nF, Capacitor_THT:C_Disc_D5.0mm_W2.5mm_P2.50mm, F.Cu at (133.5, 69.9)
- added C2: 10uF_63V, Capacitor_THT:CP_Radial_D5.0mm_P2.00mm, F.Cu at (93.5, 56.7)
- added C3: 10nF, Capacitor_THT:C_Disc_D5.0mm_W2.5mm_P2.50mm, F.Cu at (137.5, 69.9)
- added C4: 100nF, Capacitor_THT:C_Disc_D5.0mm_W2.5mm_P2.50mm, F.Cu at (141.6, 69.9)
- added C5: 100nF, Capacitor_THT:C_Disc_D5.0mm_W2.5mm_P2.50mm, F.Cu at (145.6, 69.9)
- added C6: 100nF, Capacitor_THT:C_Disc_D5.0mm_W2.5mm_P2.50mm, F.Cu at (149.7, 69.9)
- added C7: 100nF, Capacitor_THT:C_Disc_D5.0mm_W2.5mm_P2.50mm, F.Cu at (124.6, 86.7)
- added D1: LED, LED_THT:LED_D3.0mm, F.Cu at (87.0, 41.1)
- added D2: LED, LED_THT:LED_D3.0mm, F.Cu at (92.5, 41.1)
- added D3: LED, LED_THT:LED_D3.0mm, F.Cu at (98.0, 41.1)
- added D4: LED, LED_THT:LED_D3.0mm, F.Cu at (103.5, 41.1)
- added DZ1: 1N4728A, PCM_Diode_THT_AKL:D_DO-41_SOD81_P10.16mm_Horizontal_Zener, F.Cu at (139.3, 112.0)
- added DZ2: 1N4728A, PCM_Diode_THT_AKL:D_DO-41_SOD81_P10.16mm_Horizontal_Zener, F.Cu at (174.3, 100.3)
- added L1: 1.0uH, PCM_SparkFun-Coil:0805, F.Cu at (83.0, 41.6)
- added R3: 100ohm, Resistor_THT:R_Axial_DIN0207_L6.3mm_D2.5mm_P10.16mm_Horizontal, F.Cu at (170.3, 37.1)
- added R36: 2, PCM_fab:R_1206, F.Cu at (69.5, 40.1)
- added R37: 4.7k, Resistor_THT:R_Axial_DIN0207_L6.3mm_D2.5mm_P10.16mm_Horizontal, F.Cu at (133.7, 138.0)
- added R38: 4.7k, Resistor_THT:R_Axial_DIN0207_L6.3mm_D2.5mm_P10.16mm_Horizontal, F.Cu at (143.8, 144.0)
- added R39: 20k, Resistor_THT:R_Axial_DIN0207_L6.3mm_D2.5mm_P10.16mm_Horizontal, F.Cu at (187.3, 139.0)
- added R40: 20k, Resistor_THT:R_Axial_DIN0207_L6.3mm_D2.5mm_P10.16mm_Horizontal, F.Cu at (181.3, 138.8)
- added R41: 20k, Resistor_THT:R_Axial_DIN0207_L6.3mm_D2.5mm_P10.16mm_Horizontal, F.Cu at (175.3, 149.1)
- added R6: 100ohm, Resistor_THT:R_Axial_DIN0207_L6.3mm_D2.5mm_P10.16mm_Horizontal, F.Cu at (205.0, 49.0)
- added SW7: SW_Push, Button_Switch_SMD:SW_Tactile_SPST_NO_Straight_CK_PTS636Sx25SMTRLFS, F.Cu at (195.6, 71.5)
- added SW8: SW_Push, Button_Switch_SMD:SW_Tactile_SPST_NO_Straight_CK_PTS636Sx25SMTRLFS, F.Cu at (135.1, 88.8)
- added TP13: 0.5mm, PCM_SparkFun-Connector:TestPoint-0.5mm, F.Cu at (61.2, 77.8)
- added TP16: 0.5mm, PCM_SparkFun-Connector:TestPoint-0.5mm, F.Cu at (61.2, 82.6)
- added U6: INA226, Package_SO:TSSOP-10_3x3mm_P0.5mm, F.Cu at (128.7, 134.5)
- C10, C23, C25, C26, C30, C32: value 100nF_Ceramic -> 100nF
- C12: value 0.1uF_0603_16V -> 1uF_50V; footprint PCM_4ms_Capacitor:C_0603 -> Capacitor_THT:CP_Radial_D4.0mm_P1.50mm
- C14: value 0.1uF -> 22uF; footprint PCM_SparkFun-Capacitor:C_0603_1608Metric -> Capacitor_THT:CP_Radial_D5.0mm_P2.00mm
- C15: value 100nF_0603_16V -> 1uF; footprint Capacitor_SMD:C_0603_1608Metric -> Capacitor_THT:CP_Radial_D4.0mm_P1.50mm
- C16: value 100nF_0603_16V -> 10nF; footprint Capacitor_SMD:C_0603_1608Metric -> Capacitor_THT:C_Disc_D5.0mm_W2.5mm_P2.50mm
- C17, C18, C19: value 100nF_0603_16V -> 10uF_16V; footprint Capacitor_SMD:C_0603_1608Metric -> Capacitor_THT:CP_Radial_D5.0mm_P2.00mm
- C20: value 10nF_0603_25V -> 100nF; footprint Capacitor_SMD:C_0603_1608Metric -> Capacitor_THT:C_Disc_D5.0mm_W2.5mm_P2.50mm
- C21: value 10nF_0603_25V -> 22uF; footprint Capacitor_SMD:C_0603_1608Metric -> Capacitor_THT:CP_Radial_D5.0mm_P2.00mm
- C22: value 1uF_0603_25V -> 22uF; footprint Capacitor_SMD:C_0603_1608Metric -> Capacitor_THT:CP_Radial_D5.0mm_P2.00mm
- C24, C9: value 10uF_16V -> 10uF
- C27: value 10 uF -> 100nF; footprint Capacitor_SMD:C_1206_3216Metric -> Capacitor_THT:C_Disc_D5.0mm_W2.5mm_P2.50mm
- J10, J4, J5, J6: footprint Components_Footprint:POMONA_73096-2 -> MountingHole:MountingHole_4.3mm_M4_Pad_Via
- R10, R4: value 100 -> 100ohm; footprint PCM_SparkFun-Resistor:R_0603_1608Metric -> Resistor_THT:R_Axial_DIN0207_L6.3mm_D2.5mm_P10.16mm_Horizontal
- R11, R12, R13: value 4.7k -> 20k; footprint PCM_SparkFun-Resistor:R_0603_1608Metric -> Resistor_THT:R_Axial_DIN0207_L6.3mm_D2.5mm_P10.16mm_Horizontal
- R14, R5: value 10 -> 10R_0.5W; footprint PCM_SparkFun-Resistor:R_1206_3216Metric -> Resistor_THT:R_Axial_DIN0309_L9.0mm_D3.2mm_P15.24mm_Horizontal
- R25: value 1.5k_0603 -> 360R_1W; footprint Capacitor_SMD:C_0603_1608Metric -> Resistor_THT:R_Axial_DIN0414_L11.9mm_D4.5mm_P20.32mm_Horizontal
- R28: value 2Ω -> 4.7k; footprint Resistor_SMD:R_1206_3216Metric -> Resistor_THT:R_Axial_DIN0207_L6.3mm_D2.5mm_P10.16mm_Horizontal
- R32: value 100 -> 33R_1%_2512; footprint PCM_SparkFun-Resistor:R_0603_1608Metric -> PCM_Resistor_SMD_AKL:R_2512_6332Metric
- R34: value 100 -> 1.5k; footprint PCM_SparkFun-Resistor:R_0603_1608Metric -> Resistor_THT:R_Axial_DIN0207_L6.3mm_D2.5mm_P10.16mm_Horizontal
- U3: value CH340C -> CH340G
- moved J3 172.0 mm to (53.8, 41.1), turned to -90 degrees
- moved R2 166.5 mm to (57.5, 38.4), turned to 180 degrees
- moved R1 163.8 mm to (57.6, 43.9), turned to 180 degrees
- moved FB1 155.9 mm to (76.5, 61.6), turned to 180 degrees
- moved TP10 152.8 mm to (46.3, 126.3)
- moved TP11 152.8 mm to (46.3, 127.9)
- moved TP12 152.8 mm to (46.3, 129.5)
- moved TP7 152.8 mm to (46.3, 121.4)
- moved TP8 152.8 mm to (46.3, 123.0)
- moved TP9 152.8 mm to (46.3, 124.6)
- moved TP21 150.3 mm to (49.5, 123.0)
- moved C17 146.0 mm to (65.0, 40.1), turned to 180 degrees
- moved C25 146.0 mm to (46.0, 64.9), turned to 90 degrees
- moved TP22 141.3 mm to (72.0, 35.6)
- moved TP2 138.4 mm to (58.0, 79.4)
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Connections:
- C14 pad 1: IN+ -> 5V
- C14 pad 2: IN- -> GND
- C15 pad 1: /TFT_RST -> 3.3VD
- C16 pad 1: 3.3VD -> GND
- C16 pad 2: GND -> 3.3VA
- C17 pad 1: 3.3VD -> Net-(C17-Pad1)
- C18 pad 1: 3.3VD -> /VBUS
- C19 pad 1: 3.3VD -> /BAT
- C20 pad 1: 3.3VD -> IN-
- C20 pad 2: GND -> IN+
- C21 pad 1: GND -> 5V
- C21 pad 2: 3.3VA -> GND
- C22 pad 1: 3.3VD -> 5V
- C27 pad 1: Net-(C27-Pad1) -> GND
- C27 pad 2: GND -> 3.3VD
- R10 pad 1: /EC_B -> Net-(C31-Pad2)
- R10 pad 2: Net-(C28-Pad2) -> /RANGE
- R11 pad 1: /SDA1 -> AC_L
- R11 pad 2: 3.3VD -> Net-(R11-Pad2)
- R12 pad 1: /SCL1 -> Net-(R11-Pad2)
- R12 pad 2: 3.3VD -> Net-(R12-Pad2)
- R13 pad 1: 3.3VD -> Net-(R12-Pad2)
- R13 pad 2: Net-(U2-~{Alert}) -> Net-(R13-Pad2)
- R14 pad 1: Net-(R14-Pad1) -> IN-
- R14 pad 2: IN- -> Net-(R14-Pad2)
- R15_Shunt1 pad 1: Net-(R14-Pad1) -> Net-(R14-Pad2)
- R25 pad 1: 3.3VD -> Net-(C11-Pad1)
- R25 pad 2: /USB_C+ -> Net-(R24-Pad1)
- R28 pad 1: /VBUS -> /SDA1
- R28 pad 2: Net-(C27-Pad1) -> 3.3VD
- R32 pad 1: Net-(C30-Pad2) -> Net-(C8-Pad1)
- R32 pad 2: /PUSH -> Net-(J1-Pad2)
- R34 pad 1: Net-(C31-Pad2) -> /USB_C+
- R34 pad 2: /RANGE -> 3.3VD
- R4 pad 1: /EC_A -> Net-(C28-Pad2)
- R4 pad 2: Net-(C29-Pad2) -> /EC_B
- T1 pad 1: Net-(R16-Pad2) -> Net-(R13-Pad2)
- TP8 pad 1: Net-(R14-Pad1) -> Net-(R14-Pad2)

Commit message: update 16/07/2026
Parts:
- removed C11, C8: 10uF_16V, Capacitor_THT:CP_Radial_D5.0mm_P2.00mm
- removed C12: 1uF_50V, Capacitor_THT:CP_Radial_D4.0mm_P1.50mm
- removed C14, C21, C22: 22uF, Capacitor_THT:CP_Radial_D5.0mm_P2.00mm
- removed C15: 1uF, Capacitor_THT:CP_Radial_D4.0mm_P1.50mm
- removed C16: 10nF, Capacitor_THT:C_Disc_D5.0mm_W2.5mm_P2.50mm
- removed C20, C27, C30, C32: 100nF, Capacitor_THT:C_Disc_D5.0mm_W2.5mm_P2.50mm
- removed C28, C29, C31: 100nF_Ceramic, Capacitor_THT:C_Disc_D5.0mm_W2.5mm_P2.50mm
- removed D1, D2, D3, D4: LED, LED_THT:LED_D3.0mm
- removed R10, R3, R4, R6: 100ohm, Resistor_THT:R_Axial_DIN0207_L6.3mm_D2.5mm_P10.16mm_Horizontal
- removed R39, R40, R41: 20k, Resistor_THT:R_Axial_DIN0207_L6.3mm_D2.5mm_P10.16mm_Horizontal
- added C13: 10uF, PCM_SparkFun-Capacitor:C_0805_2012Metric, B.Cu at (132.2, 36.5)
- added C34: 10uF, PCM_SparkFun-Capacitor:C_0805_2012Metric, B.Cu at (134.2, 41.5)
- added C36: 10uF, PCM_SparkFun-Capacitor:C_0805_2012Metric, B.Cu at (138.0, 59.9)
- added C37: 10uF, PCM_SparkFun-Capacitor:C_0805_2012Metric, B.Cu at (136.8, 55.0)
- added C38: 10uF, PCM_SparkFun-Capacitor:C_0805_2012Metric, B.Cu at (150.1, 35.4)
- added C39: 10uF, PCM_SparkFun-Capacitor:C_0805_2012Metric, B.Cu at (150.1, 32.4)
- added C40: 10uF, PCM_SparkFun-Capacitor:C_0805_2012Metric, B.Cu at (118.3, 87.8)
- added C41: 10uF, PCM_SparkFun-Capacitor:C_0805_2012Metric, F.Cu at (134.1, 128.1)
- added C42: 100nF_1206_10%, Components_Footprint:CAPC3216X100N, F.Cu at (111.6, 116.0)
- added C43: 100nF_1206_10%, Components_Footprint:CAPC3216X100N, F.Cu at (140.7, 65.5)
- added C44: 100nF_1206, Components_Footprint:CAPC3216X100N, F.Cu at (143.2, 65.5)
- added C45: 100nF_1206_10%, Components_Footprint:CAPC3216X100N, F.Cu at (135.7, 65.4)
- added C46: 100nF_1206_10%, Components_Footprint:CAPC3216X100N, F.Cu at (138.2, 65.4)
- added C47: 100nF_1206_10%, Components_Footprint:CAPC3216X100N, F.Cu at (132.0, 77.3)
- added C48: 100nF_1206_10%, Components_Footprint:CAPC3216X100N, F.Cu at (135.7, 81.4)
- added D5: Blue, PCM_SparkFun-LED:LED_1206_3216Metric_Blue, B.Cu at (139.2, 40.6)
- added D6: Blue, PCM_SparkFun-LED:LED_1206_3216Metric_Blue, B.Cu at (139.2, 37.3)
- added D7: Blue, PCM_SparkFun-LED:LED_1206_3216Metric_Blue, B.Cu at (139.2, 34.0)
- added D8: Blue, PCM_SparkFun-LED:LED_1206_3216Metric_Blue, B.Cu at (139.2, 30.7)
- added R16: 4.7k_0805, Components_Footprint:RESC2012X60N, F.Cu at (117.1, 123.5)
- added R17: 4.7k_0805, Components_Footprint:RESC2012X60N, F.Cu at (117.1, 121.5)
- added R18: 4.7k_0805, Components_Footprint:RESC2012X60N, F.Cu at (117.1, 119.5)
- added R19: 10k_1206, PCM_fab:R_1206, F.Cu at (132.0, 72.3)
- added R20: 10k_1206, PCM_fab:R_1206, F.Cu at (140.7, 81.4)
- added R21: 10k_1206, PCM_fab:R_1206, F.Cu at (129.2, 66.1)
- added R42: 10k_1206, PCM_fab:R_1206, F.Cu at (163.3, 108.6)
- C1: value 100nF -> 1uF_1206; footprint Capacitor_THT:C_Disc_D5.0mm_W2.5mm_P2.50mm -> Components_Footprint:CAPC3216X180N
- C10: value 100nF -> 100nF_1206_10%; footprint Capacitor_THT:C_Disc_D5.0mm_W2.5mm_P2.50mm -> Components_Footprint:CAPC3216X100N; moved to B.Cu
- C17: value 10uF_16V -> 100nF_1206_10%; footprint Capacitor_THT:CP_Radial_D5.0mm_P2.00mm -> Components_Footprint:CAPC3216X100N; moved to B.Cu
- C18, C19: value 10uF_16V -> 100nF_1206_10%; footprint Capacitor_THT:CP_Radial_D5.0mm_P2.00mm -> Components_Footprint:CAPC3216X100N
- C2: value 10uF_63V -> 1uF_1206; footprint Capacitor_THT:CP_Radial_D5.0mm_P2.00mm -> Components_Footprint:CAPC3216X180N; moved to B.Cu
- C23, C25, C26: value 100nF -> 100nF_1206_10%; footprint Capacitor_THT:C_Disc_D5.0mm_W2.5mm_P2.50mm -> Components_Footprint:CAPC3216X100N
- C24: value 10uF -> 100nF_1206_10%; footprint Capacitor_THT:CP_Radial_D5.0mm_P2.00mm -> Components_Footprint:CAPC3216X100N
- C3: value 10nF -> 22uF; footprint Capacitor_THT:C_Disc_D5.0mm_W2.5mm_P2.50mm -> PCM_SparkFun-Capacitor:C_1206_3216Metric; moved to B.Cu
- C4: value 100nF -> 10nF_1206; footprint Capacitor_THT:C_Disc_D5.0mm_W2.5mm_P2.50mm -> Components_Footprint:CAPC3216X90N
- C5: value 100nF -> 10nF_1206; footprint Capacitor_THT:C_Disc_D5.0mm_W2.5mm_P2.50mm -> Components_Footprint:CAPC3216X90N; moved to B.Cu
- C6, C7: value 100nF -> 22uF; footprint Capacitor_THT:C_Disc_D5.0mm_W2.5mm_P2.50mm -> PCM_SparkFun-Capacitor:C_1206_3216Metric; moved to B.Cu
- C9: value 10uF -> 100nF_1206_10%; footprint Capacitor_THT:CP_Radial_D5.0mm_P2.00mm -> Components_Footprint:CAPC3216X100N; moved to B.Cu
- DZ1, FB1, J1, J3, J9, L1, R1, R2, R32, R35, R36, SW6, TP14, TP15, TP17, TP22, TP23, TP24, TP4, TP5, TP6, U4, U5: moved to B.Cu
- R11, R12, R13: value 20k -> 20k_1206_1%; footprint Resistor_THT:R_Axial_DIN0207_L6.3mm_D2.5mm_P10.16mm_Horizontal -> Components_Footprint:RESC3216X70N
- R15, R26, R29: value 10k -> 20k_1206_1%; footprint Resistor_THT:R_Axial_DIN0207_L6.3mm_D2.5mm_P10.16mm_Horizontal -> Components_Footprint:RESC3216X70N
- R22, R23: value 470k -> 100R_1206; footprint Resistor_THT:R_Axial_DIN0207_L6.3mm_D2.5mm_P10.16mm_Horizontal -> PCM_fab:R_1206
- R24: value 1k -> 100R_1206; footprint Resistor_THT:R_Axial_DIN0207_L6.3mm_D2.5mm_P10.16mm_Horizontal -> PCM_fab:R_1206
- R25: value 360R_1W -> 100R_1206; footprint Resistor_THT:R_Axial_DIN0414_L11.9mm_D4.5mm_P20.32mm_Horizontal -> PCM_fab:R_1206
- R27, R30: value 10k -> 470k_1206; footprint Resistor_THT:R_Axial_DIN0207_L6.3mm_D2.5mm_P10.16mm_Horizontal -> PCM_fab:R_1206; moved to B.Cu
- R28, R37, R38: value 4.7k -> 10k_1206; footprint Resistor_THT:R_Axial_DIN0207_L6.3mm_D2.5mm_P10.16mm_Horizontal -> PCM_fab:R_1206
- R31, R33: value 10k -> 470k_1206; footprint Resistor_THT:R_Axial_DIN0207_L6.3mm_D2.5mm_P10.16mm_Horizontal -> PCM_fab:R_1206
- R7: value 470k -> 1k_2512; footprint Resistor_THT:R_Axial_DIN0207_L6.3mm_D2.5mm_P10.16mm_Horizontal -> PCM_Resistor_SMD_AKL:R_2512_6332Metric; moved to B.Cu
- R8: value 470k -> 1k_2512; footprint Resistor_THT:R_Axial_DIN0207_L6.3mm_D2.5mm_P10.16mm_Horizontal -> PCM_Resistor_SMD_AKL:R_2512_6332Metric
- R9: value 1k -> 360_1206; footprint Resistor_THT:R_Axial_DIN0207_L6.3mm_D2.5mm_P10.16mm_Horizontal -> Components_Footprint:RESC3116X65N
- moved R31 120.3 mm to (133.5, 133.8), turned to 0 degrees
- moved C18 112.9 mm to (165.9, 108.6), turned to 90 degrees
- moved TP13 112.0 mm to (160.7, 129.2), turned to 180 degrees
- moved TP16 108.0 mm to (160.7, 124.7)
- moved C24 106.7 mm to (150.9, 100.1), turned to 180 degrees
- moved C19 96.7 mm to (174.3, 92.1), turned to 90 degrees
- moved R29 96.4 mm to (161.0, 120.7)
- moved TP2 96.0 mm to (137.2, 133.7), turned to 180 degrees
- moved TP17 95.7 mm to (147.5, 57.5), turned to 90 degrees
- moved J9 92.5 mm to (139.8, 25.5), turned to 0 degrees
- moved U4 91.3 mm to (147.1, 41.5), turned to -90 degrees
- moved R33 90.8 mm to (133.5, 130.8)
- moved C25 90.5 mm to (120.6, 116.0), turned to -90 degrees
- moved TP19 88.3 mm to (150.2, 83.0), turned to 180 degrees
- moved TP20 87.4 mm to (153.0, 83.0), turned to 180 degrees
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Connections:
- C1 pad 1: GND -> 3.3VD
- C1 pad 2: 3.3VD -> GND
- C10 pad 1: GND -> 5V
- C10 pad 2: 3.3VD -> GND
- C17 pad 1: Net-(C17-Pad1) -> 3.3VA
- C18 pad 1: /VBUS -> Net-(C18-Pad1)
- C19 pad 1: /BAT -> Net-(C19-Pad1)
- C2 pad 1: Net-(C2-Pad1) -> 3.3VD
- C23 pad 1: GND -> Net-(C23-Pad1)
- C23 pad 2: 3.3VA -> GND
- C24 pad 1: 5V -> Net-(C24-Pad1)
- C25 pad 1: GND -> 3.3VD
- C25 pad 2: 5V -> GND
- C26 pad 1: GND -> 3.3VD
- C26 pad 2: 3.3VD -> GND
- C3 pad 1: GND -> 5V
- C3 pad 2: 3.3VD -> GND
- C4 pad 1: GND -> 3.3VD
- C4 pad 2: 3.3VD -> GND
- C5 pad 1: GND -> 3.3VA
- C5 pad 2: 3.3VD -> GND
- C6 pad 1: GND -> 5V
- C6 pad 2: 3.3VD -> GND
- C7 pad 1: GND -> 5V
- C7 pad 2: /TFT_RST -> GND
- J1 pad 1: Net-(C8-Pad1) -> Net-(C40-Pad1)
- R12 pad 1: Net-(R11-Pad2) -> AC_N
- R15 pad 1: 3.3VD -> Net-(R11-Pad2)
- R15 pad 2: /TFT_RST -> Net-(R15-Pad2)
- R22 pad 1: Net-(C11-Pad1) -> /EC_A
- R22 pad 2: 3.3VA -> Net-(C23-Pad1)
- R23 pad 1: GND -> Net-(C24-Pad1)
- R23 pad 2: Net-(C11-Pad1) -> /EC_B
- R24 pad 1: Net-(R24-Pad1) -> Net-(C19-Pad1)
- R24 pad 2: ADC2 -> /PUSH
- R25 pad 1: Net-(C11-Pad1) -> Net-(C18-Pad1)
- R25 pad 2: Net-(R24-Pad1) -> /RANGE
- R26 pad 1: Net-(SW3-B) -> Net-(R15-Pad2)
- R26 pad 2: Net-(U1-BOOT0) -> Net-(R26-Pad2)
- R27 pad 1: GND -> 3.3VA
- R27 pad 2: Net-(U1-PB2) -> Net-(C40-Pad1)
- R28 pad 1: /SDA1 -> 3.3VD
- R28 pad 2: 3.3VD -> Net-(C23-Pad1)
- R29 pad 1: 3.3VD -> Net-(R13-Pad2)
- R29 pad 2: Net-(C29-Pad2) -> Net-(R29-Pad2)
- R30 pad 1: 3.3VD -> Net-(C40-Pad1)
- R30 pad 2: Net-(C28-Pad2) -> GND
- R31 pad 1: 3.3VD -> 3.3VA
- R31 pad 2: Net-(C30-Pad2) -> Net-(C41-Pad1)
- R32 pad 1: Net-(C8-Pad1) -> Net-(C40-Pad1)
- R33 pad 1: 3.3VD -> GND
- R33 pad 2: Net-(C31-Pad2) -> Net-(C41-Pad1)
- R35 pad 2: Net-(C2-Pad1) -> Net-(C36-Pad1)
- R36 pad 2: Net-(C17-Pad1) -> Net-(C13-Pad1)
- R37 pad 1: /SCL1 -> 3.3VD
- R37 pad 2: 3.3VD -> Net-(C24-Pad1)
- R38 pad 2: Net-(U6-~{Alert}) -> Net-(C19-Pad1)
- R7 pad 1: Net-(C8-Pad1) -> ADC1
- R7 pad 2: 3.3VA -> Net-(J1-Pad2)
- R8 pad 1: GND -> Net-(R8-Pad1)
- R8 pad 2: Net-(C8-Pad1) -> ADC2
- R9 pad 1: Net-(J1-Pad2) -> Net-(C41-Pad1)
- R9 pad 2: ADC1 -> Net-(R8-Pad1)
- SW4 pad A: Net-(C29-Pad2) -> Net-(C23-Pad1)
- SW4 pad B: Net-(C28-Pad2) -> Net-(C24-Pad1)
- SW4 pad D: Net-(C30-Pad2) -> Net-(C19-Pad1)
- SW7 pad 2: Net-(C31-Pad2) -> Net-(C18-Pad1)
- T1 pad 1: Net-(R13-Pad2) -> Net-(R26-Pad2)
- T1 pad 2: Net-(R41-Pad2) -> Net-(R29-Pad2)
- T1 pad 3: Net-(R24-Pad1) -> Net-(R8-Pad1)
- T1 pad 4: Net-(C11-Pad1) -> Net-(C41-Pad1)
- TP13 pad 1: Net-(R13-Pad2) -> Net-(R26-Pad2)
- TP16 pad 1: Net-(R41-Pad2) -> Net-(R29-Pad2)
- TP2 pad 1: Net-(C11-Pad1) -> Net-(C41-Pad1)
- TP5 pad 1: Net-(C8-Pad1) -> Net-(C40-Pad1)
Other:
- board outline added: 82 x 120 mm
