File: Energy_Meter.kicad_pcb (KiCad board)
At the start: 2 copper layers, 98 x 97.5 mm, 119 parts, among them J1 Conn_Jack_Stereo_3.5mm_SMD_RA, J10 Conn_01x01, J2 Conn_01x04_Pin, J3 USB_C_Receptacle, J4 Conn_01x01, J5 Conn_01x01, J6 Conn_01x01, J9 3.5mm, SW4 EC11E15244G1, SW6 SW_Push, SW7 SW_Push, SW8 SW_Push, T1 ZMPT101B, U1 STM32F103C8Tx, U3 CH340G, U4 AMS1117-3.3, U5 IP5306, U6 INA226, X1 SMD5032-4

Commit message: update 20/07/2026
Parts:
- removed R15, R26, R29: 20k_1206_1%, Components_Footprint:RESC3216X70N
- added R10: 20k_1206, Components_Footprint:RES_ERA8ARB203V, F.Cu at (113.2, 117.8)
- added R14: 20k_1206, Components_Footprint:RES_ERA8ARB203V, F.Cu at (122.1, 133.2)
- added R5: 20k_1206, Components_Footprint:RES_ERA8ARB203V, F.Cu at (102.7, 117.8)
- added TP18: 0.5mm, PCM_SparkFun-Connector:TestPoint-0.5mm, F.Cu at (147.1, 105.3)
- added TP25: 0.5mm, PCM_SparkFun-Connector:TestPoint-0.5mm, F.Cu at (145.7, 107.2)
- added TP26: 0.5mm, PCM_SparkFun-Connector:TestPoint-0.5mm, B.Cu at (159.0, 93.0)
- added TP27: 0.5mm, PCM_SparkFun-Connector:TestPoint-0.5mm, B.Cu at (177.6, 98.7)
- J10, J4, J5, J6: footprint MountingHole:MountingHole_4.3mm_M4_Pad_Via -> MountingHole:MountingHole_4.3mm_M4_Pad
- R11, R12, R13: value 20k_1206_1% -> 20k_1206; footprint Components_Footprint:RESC3216X70N -> Components_Footprint:RES_ERA8ARB203V
- moved R11 22.5 mm to (122.2, 117.6)
- moved TP16 12.7 mm to (125.5, 132.9)
- moved C41 12.7 mm to (149.9, 123.2)
- moved R31 12.7 mm to (149.9, 118.2)
- moved R33 12.7 mm to (149.9, 120.7)
- moved R9 12.7 mm to (147.5, 126.7)
- moved TP1 12.7 mm to (153.9, 126.0)
- moved D5 12.7 mm to (152.9, 128.3)
- moved R8 12.7 mm to (150.4, 131.9)
- moved T1 12.7 mm to (136.2, 125.8)
- moved TP13 12.7 mm to (125.6, 118.9)
- moved TP2 12.7 mm to (146.9, 118.2)
- moved R13 8.82 mm to (113.2, 133.0)
- moved C19 5.54 mm to (178.0, 106.2)
- moved R23 5.54 mm to (152.5, 110.4)
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Connections:
- R11 pad 1: AC_L -> Net-(R10-Pad2)
- T1 pad 1: Net-(R26-Pad2) -> Net-(R11-Pad2)
- TP13 pad 1: Net-(R26-Pad2) -> Net-(R11-Pad2)
Routing:
- net ADC2: track 16.3 -> 42.7 mm
- net 3.3VA: track 124.6 -> 149.3 mm
- net Net-(R26-Pad2): track 7.69 -> 0.00 mm
- net Net-(R10-Pad1): track 0.00 -> 6.47 mm
- net /PUSH: track 39.7 -> 33.8 mm
- net 3.3VD: track 391.5 -> 385.7 mm
- net /EC_B: track 23.1 -> 17.5 mm
- net Net-(R11-Pad2): track 1.94 -> 7.50 mm
- net Net-(R12-Pad2): track 1.94 -> 7.37 mm
- net Net-(R10-Pad2): track 0.00 -> 5.15 mm
- net /EC_A: track 17.6 -> 12.7 mm
- net GND: track 114.5 -> 118.3 mm, vias 0 -> 8
- net AC_L: track 6.47 -> 10.3 mm
- net Net-(R13-Pad2): track 1.94 -> 4.90 mm
- net AC_N: track 6.50 -> 9.25 mm
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- added copper zone on B.Cu, net GND
- added copper zone on F.Cu, net GND
Other:
- outline, holes or cut-outs redrawn

Commit message: update 22/07/2026
Parts:
- added R20: 4.7k_0805, Components_Footprint:RESC2012X60N, F.Cu at (140.1, 44.3)
- added R26: 4.7k_0805, Components_Footprint:RESC2012X60N, F.Cu at (137.5, 44.3)
- DS1: value 4311 -> OLED_128X64_1.3_I2C; footprint Components_Footprint:MODULE_4311 -> Components_Footprint:LCD_OLED_128X64_1.3_I2C
- moved C24 17.9 mm to (133.6, 45.0), turned to 0 degrees
- moved TP17 11.1 mm to (151.9, 55.6)
- moved TP14 8.71 mm to (112.6, 48.6)
- moved DS1 3.92 mm to (136.3, 63.4), turned to 0 degrees
- moved J4 1.39 mm to (92.1, 117.8)
- moved J10 1.20 mm to (91.9, 132.5)
Connections:
- DS1 pad 2: unconnected-(DS1-3VO-Pad2) -> GND
- DS1 pad 3: GND -> /SCL2
- DS1 pad 4: /TFT_SCK -> /SDA2
- U1 pad 19: /TFT_BLK -> unconnected-(U1-PB1-Pad19)
- U1 pad 21: unconnected-(U1-PB10-Pad21) -> /SCL2
- U1 pad 22: unconnected-(U1-PB11-Pad22) -> /SDA2
- U1 pad 26: /TFT_SCK -> unconnected-(U1-PB13-Pad26)
- U1 pad 27: /TFT_MISO -> unconnected-(U1-PB14-Pad27)
- U1 pad 28: /TFT_MOSI -> unconnected-(U1-PB15-Pad28)
- U1 pad 45: /TFT_CS -> unconnected-(U1-PB8-Pad45)
- U1 pad 46: /TFT_DC -> unconnected-(U1-PB9-Pad46)
Routing:
- net /TFT_SCK: track 85.1 -> 0.00 mm, vias 2 -> 0
- net /TFT_MISO: track 81.5 -> 0.00 mm, vias 2 -> 0
- net /TFT_MOSI: track 77.7 -> 0.00 mm, vias 2 -> 0
- net /TFT_BLK: track 63.5 -> 0.00 mm, vias 2 -> 0
- net /SCL2: track 0.00 -> 62.6 mm, vias 0 -> 2
- net /SDA2: track 0.00 -> 61.0 mm, vias 0 -> 2
- net /TFT_CS: track 59.8 -> 0.00 mm, vias 2 -> 0
- net /TFT_DC: track 53.2 -> 0.00 mm, vias 2 -> 0
- net /TFT_RST: track 72.7 -> 36.4 mm, vias 3 -> 2
- net unconnected-(U1-PB1-Pad19): track 0.00 -> 35.6 mm, vias 0 -> 2
- net 3.3VD: track 385.7 -> 358.4 mm, vias 8 -> 11
- net GND: track 118.3 -> 112.4 mm
- net AC_L: track 10.3 -> 8.85 mm
- net AC_N: track 9.25 -> 8.59 mm

Commit message: update 27/07/2026
Parts:
- removed TP12: 0.5mm, PCM_SparkFun-Connector:TestPoint-0.5mm
- moved D6 6.98 mm to (108.2, 96.8)
- moved TP4 5.18 mm to (109.4, 95.1), turned to 0 degrees
- moved J6 2.01 mm to (91.1, 62.8)
- moved J5 1.90 mm to (91.1, 81.5)
- moved R20 1.57 mm to (141.3, 45.2), turned to 0 degrees
- moved J4 1.55 mm to (93.7, 118.1)
- moved TP6 1.13 mm to (87.5, 102.5)
- moved J10 1.11 mm to (93.0, 132.7)
- moved R7 1.04 mm to (105.7, 100.2)
- moved C43 1.04 mm to (87.2, 100.0)
- moved J1 1.04 mm to (98.4, 92.3)
- moved R27 1.04 mm to (92.2, 100.5)
- moved R30 1.04 mm to (89.7, 100.5)
- moved TP5 1.04 mm to (89.9, 96.8)
- moved R32 1.04 mm to (97.5, 100.2)
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Connections:
- C26 pad 1: IN+ -> Net-(U6-Vin+)
- C26 pad 2: IN- -> Net-(U6-Vbus)
- R15_Shunt1 pad 1: Net-(R15_Shunt1-Pad1) -> IN-
- R15_Shunt1 pad 2: Net-(R15_Shunt1-Pad2) -> IN+
- R4 pad 1: IN- -> Net-(U6-Vbus)
- R4 pad 2: Net-(R15_Shunt1-Pad1) -> IN-
- R6 pad 1: Net-(R15_Shunt1-Pad2) -> IN+
- R6 pad 2: IN+ -> Net-(U6-Vin+)
- TP7 pad 1: Net-(R15_Shunt1-Pad2) -> IN+
- TP8 pad 1: Net-(R15_Shunt1-Pad1) -> IN-
- U6 pad 10: IN+ -> Net-(U6-Vin+)
- U6 pad 8: IN- -> Net-(U6-Vbus)
- U6 pad 9: IN- -> Net-(U6-Vbus)
Routing:
- net unconnected-(U1-PB1-Pad19): track 35.6 -> 0.00 mm, vias 2 -> 0
- net Net-(U6-Vbus): track 0.00 -> 7.36 mm
- net GND: track 112.4 -> 119.6 mm, vias 8 -> 1292
- net /VBUS: track 25.8 -> 32.9 mm, vias 0 -> 2
- net ADC1: track 48.1 -> 42.8 mm
- net Net-(U6-Vin+): track 0.00 -> 5.07 mm
- net /USB_C+: track 8.02 -> 12.6 mm, vias 0 -> 2
- net IN-: track 16.2 -> 11.6 mm
- net Net-(R15_Shunt1-Pad2): track 4.49 -> 0.00 mm
- net Net-(R15_Shunt1-Pad1): track 4.45 -> 0.00 mm
- net /USB_C-: track 8.34 -> 10.8 mm
- net IN+: track 12.8 -> 11.3 mm
- net AC_L: track 8.85 -> 7.44 mm
- net 3.3VD: track 358.4 -> 359.7 mm, vias 11 -> 10
- net AC_N: track 8.59 -> 7.43 mm
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