File: Energy_Meter.kicad_pcb (KiCad board)
At the start: 2 copper layers, 98 x 97.5 mm, 124 parts, among them J1 Conn_Jack_Stereo_3.5mm_SMD_RA, J10 Conn_01x01, J2 Conn_01x04_Pin, J3 USB_C_Receptacle, J4 Conn_01x01, J5 Conn_01x01, J6 Conn_01x01, J9 3.5mm, SW4 EC11E15244G1, SW6 SW_Push, SW7 SW_Push, SW8 SW_Push, T1 ZMPT101B, U1 STM32F103C8Tx, U3 CH340G, U4 AMS1117-3.3, U5 IP5306, U6 INA226, X1 SMD5032-4

Commit message: update 27/07/2026
Parts:
- added C28: 100nF_0805, PCM_Capacitor_SMD_AKL:C_0805_2012Metric, F.Cu at (133.6, 45.1)
- C24: moved to B.Cu
- moved C24 34.2 mm to (163.3, 61.9)
- moved TP22 0.51 mm to (166.9, 59.5)
Connections:
- R21 pad 1: 3.3VD -> GND
Routing:
- net 3.3VD: track 359.7 -> 357.3 mm

Commit message: update 29/07/2026
Parts:
- added R15: 0R_0805, PCM_Resistor_SMD_AKL:R_0805_2012Metric, F.Cu at (149.9, 83.6)
- added R29: 0R_0805, PCM_Resistor_SMD_AKL:R_0805_2012Metric, F.Cu at (147.5, 84.8)
- added R34: 0R_0805, PCM_Resistor_SMD_AKL:R_0805_2012Metric, B.Cu at (146.5, 94.2)
- added R39: 0R_0805, PCM_Resistor_SMD_AKL:R_0805_2012Metric, B.Cu at (148.9, 93.6)
- added R46: 0R_0805, PCM_Resistor_SMD_AKL:R_0805_2012Metric, F.Cu at (156.7, 92.2)
- added R47: 0R_0805, PCM_Resistor_SMD_AKL:R_0805_2012Metric, F.Cu at (156.7, 90.0)
- moved TP26 1.59 mm to (158.6, 94.6)
Connections:
- U1 pad 21: /SCL2 -> Net-(U1-PB10)
- U1 pad 22: /SDA2 -> Net-(U1-PB11)
- U1 pad 30: /TX -> Net-(U1-PA9)
- U1 pad 31: /RX -> Net-(U1-PA10)
- U1 pad 42: /SCL1 -> Net-(U1-PB6)
- U1 pad 43: /SDA1 -> Net-(U1-PB7)
Routing:
- net /RX: track 48.7 -> 40.7 mm
- net /TX: track 49.5 -> 42.5 mm
- net Net-(U1-PA10): track 0.00 -> 5.72 mm
- net Net-(U1-PB6): track 0.00 -> 5.30 mm
- net Net-(U1-PA9): track 0.00 -> 5.01 mm
- net /SDA2: track 61.1 -> 56.6 mm
- net /SDA1: track 61.2 -> 56.8 mm
- net /SCL1: track 65.3 -> 61.8 mm
- net Net-(U1-PB7): track 0.00 -> 3.30 mm
- net /SCL2: track 62.9 -> 59.8 mm
- net Net-(U1-PB10): track 0.00 -> 3.04 mm, vias 0 -> 1
- net Net-(U1-PB11): track 0.00 -> 2.58 mm, vias 0 -> 1
- net /RANGE: track 12.3 -> 11.1 mm
- net /SWCLK: track 25.7 -> 25.0 mm
- net GND: track 119.6 -> 119.3 mm, vias 1292 -> 1080

Commit message: update 29/08/2026
Parts:
- J10, J4, J5, J6: footprint MountingHole:MountingHole_4.3mm_M4_Pad -> MountingHole:MountingHole_4.5mm_Pad
- moved J1 5.65 mm to (92.8, 92.1)
- moved TP5 0.94 mm to (89.7, 97.8)
Routing:
- net Net-(C43-Pad1): track 14.3 -> 20.7 mm
- net Net-(J1-Pad2): track 17.5 -> 21.0 mm
- net GND: vias 1080 -> 1295
